File: hardware/pcb/espSFD/espSFD.kicad_pcb (KiCad board)
At the start: 2 copper layers, 68.6 x 34.3 mm, 9 parts, among them J1 Conn_01x06_Socket, J2 Conn_02x10_Odd_Even, Q1 IRLU3110Z, U1 WeMos_D1_mini, U2 TSR_1-2415

Commit message: xhd
Parts:
- H1, H2: footprint MountingHole:MountingHole_3.2mm_M3_Pad -> MountingHole:MountingHole_3.2mm_M3_DIN965_Pad
Changed lines of the file:
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@@
   (net 20 "Net-(U1-D0)")
   (net 21 "Net-(Q1-G)")
-  (footprint "MountingHole:MountingHole_3.2mm_M3_Pad" (layer "F.Cu")
+  (footprint "MountingHole:MountingHole_3.2mm_M3_DIN965_Pad" (layer "F.Cu")
     (at 106.68 93.98)
-    (descr "Mounting Hole 3.2mm, M3")
-    (tags "mounting hole 3.2mm m3")
+    (descr "Mounting Hole 3.2mm, M3, DIN965")
+    (tags "mounting hole 3.2mm m3 din965")
     (property "Sheetfile" "espSFD.kicad_sch")
     (property "Sheetname" "")
@@
     (property "ki_keywords" "mounting hole")
     (attr exclude_from_pos_files)
-    (fp_text reference "H2" (at 0 -4.2) (layer "F.SilkS") hide
-        (effects (font (size 1 1) (thickness 0.15)))
-    )
-    (fp_text value "MountingHole_Pad" (at 0 4.2) (layer "F.Fab") hide
+    (fp_text reference "H2" (at 0 -3.8) (layer "F.SilkS")
+        (effects (font (size 1 1) (thickness 0.15)))
+    )
+    (fp_text value "MountingHole_Pad" (at 0 3.8) (layer "F.Fab")
         (effects (font (size 1 1) (thickness 0.15)))
     )
@@
         (effects (font (size 1 1) (thickness 0.15)))
     )
-    (fp_circle (center 0 0) (end 3.2 0)
+    (fp_circle (center 0 0) (end 2.8 0)
       (stroke (width 0.15) (type solid)) (fill none) (layer "Cmts.User"))
-    (fp_circle (center 0 0) (end 3.45 0)
+    (fp_circle (center 0 0) (end 3.05 0)
       (stroke (width 0.05) (type solid)) (fill none) (layer "F.CrtYd"))
-    (pad "1" thru_hole circle (at 0 0) (size 6.4 6.4) (drill 3.2) (layers "*.Cu" "*.Mask")
+    (pad "1" thru_hole circle (at 0 0) (size 5.6 5.6) (drill 3.2) (layers "*.Cu" "*.Mask")
       (net 1 "GND") (pinfunction "1") (pintype "input"))
   )
@@
     )
   )
-  (footprint "MountingHole:MountingHole_3.2mm_M3_Pad" (layer "F.Cu")
+  (footprint "MountingHole:MountingHole_3.2mm_M3_DIN965_Pad" (layer "F.Cu")
     (at 85.09 93.98)
-    (descr "Mounting Hole 3.2mm, M3")
-    (tags "mounting hole 3.2mm m3")
+    (descr "Mounting Hole 3.2mm, M3, DIN965")
+    (tags "mounting hole 3.2mm m3 din965")
     (property "Sheetfile" "espSFD.kicad_sch")
     (property "Sheetname" "")
@@
     (property "ki_keywords" "mounting hole")
     (attr exclude_from_pos_files)
-    (fp_text reference "H1" (at 0 -4.2) (layer "F.SilkS") hide
-        (effects (font (size 1 1) (thickness 0.15)))
-    )
-    (fp_text value "MountingHole_Pad" (at 0 4.2) (layer "F.Fab") hide
+    (fp_text reference "H1" (at 0 -3.8) (layer "F.SilkS")
+        (effects (font (size 1 1) (thickness 0.15)))
+    )
+    (fp_text value "MountingHole_Pad" (at 0 3.8) (layer "F.Fab")
         (effects (font (size 1 1) (thickness 0.15)))
     )
@@
         (effects (font (size 1 1) (thickness 0.15)))
     )
-    (fp_circle (center 0 0) (end 3.2 0)
+    (fp_circle (center 0 0) (end 2.8 0)
       (stroke (width 0.15) (type solid)) (fill none) (layer "Cmts.User"))
-    (fp_circle (center 0 0) (end 3.45 0)
+    (fp_circle (center 0 0) (end 3.05 0)
       (stroke (width 0.05) (type solid)) (fill none) (layer "F.CrtYd"))
-    (pad "1" thru_hole circle (at 0 0) (size 6.4 6.4) (drill 3.2) (layers "*.Cu" "*.Mask")
+    (pad "1" thru_hole circle (at 0 0) (size 5.6 5.6) (drill 3.2) (layers "*.Cu" "*.Mask")
       (net 1 "GND") (pinfunction "1") (pintype "input"))
   )

Commit message: es dghdgfj fcgj
Parts:
- added JP1: SolderJumper_3_Open, Library:SolderJumper-3_P1.3mm_Open_Pad1.0x1.5mm no silk, F.Cu at (66.0, 102.9)
- added JP2: SolderJumper_3_Open, Library:SolderJumper-3_P1.3mm_Open_Pad1.0x1.5mm no silk, F.Cu at (66.0, 100.3)
- moved U1 69.6 mm to (50.8, 85.1), turned to 0 degrees
- moved R1 53.6 mm to (58.4, 87.6), turned to 0 degrees
- moved R2 40.9 mm to (66.0, 85.1), turned to 180 degrees
- moved H2 40.9 mm to (65.8, 94.0), turned to 180 degrees
- moved J1 40.7 mm to (100.3, 106.7), turned to 90 degrees
- moved J2 26.8 mm to (91.4, 82.5), turned to 0 degrees
- moved Q1 25.7 mm to (83.8, 80.3), turned to -90 degrees
- moved U2 16.5 mm to (81.3, 101.6), turned to -90 degrees
- moved H1 1.27 mm to (83.8, 94.0), turned to 180 degrees
Connections:
- J2 pad 17: RX -> TX
- J2 pad 19: TX -> RX
- U1 pad 11: RX -> RX1
- U1 pad 12: TX -> TX1
- U1 pad 15: unconnected-(U1-RX-Pad15) -> RX0
- U1 pad 16: unconnected-(U1-TX-Pad16) -> TX0
Routing:
- net TX0: track 0.00 -> 20.4 mm, vias 0 -> 1
- net RX0: track 0.00 -> 19.6 mm, vias 0 -> 1
- net TX1: track 0.00 -> 8.45 mm
- net RX1: track 0.00 -> 8.45 mm
- net Net-(Q1-G): track 17.6 -> 22.3 mm
- net Motor N: track 24.7 -> 22.1 mm
- net TX: track 34.3 -> 31.9 mm, vias 0 -> 1
- net Motor L: track 25.7 -> 23.8 mm
- net RX: track 32.1 -> 30.4 mm, vias 0 -> 1
- net En Motor: track 36.1 -> 34.5 mm
- net GND: vias 4 -> 64
Other:
- board size 68.6 x 34.3 mm -> 69 x 35 mm
- board text added: "0"
- board text added: "1"
- board text added: "Bus"
- board text added: "RX"
- board text added: "RX0"
- board text added: "RX1"
- board text added: "TX"
- board text added: "TX0"
- board text added: "TX1"

Commit message: vcb
Signed-off-by: Christian Backus <chrissileinus@googlemail.com>
Parts:
- removed H1, H2: MountingHole_Pad, MountingHole:MountingHole_3.2mm_M3_DIN965_Pad
- added DRA1: DIN_Rail_Adapter, Library:DINRailAdapter_3xM3_PhoenixContact_1201578, F.Cu at (70.3, 106.5)
- added DRA2: DIN_Rail_Adapter, Library:DINRailAdapter_3xM3_PhoenixContact_1201578, F.Cu at (70.3, 81.5)
- moved R2 9.16 mm to (71.1, 92.7)
- moved Q1 8.18 mm to (80.3, 87.6), turned to 0 degrees
- moved U2 7.62 mm to (81.3, 94.0)
- moved R1 5.68 mm to (63.5, 90.2)
- moved JP1 2.56 mm to (66.0, 100.3)
- moved JP2 2.55 mm to (66.0, 97.8)
Routing:
- net Net-(Q1-G): track 22.3 -> 12.7 mm
- net Net-(U1-D0): track 8.67 -> 12.7 mm
- net En Motor: track 34.5 -> 37.9 mm
- net TX0: track 20.4 -> 18.6 mm
- net RX1: track 8.45 -> 7.40 mm
- net RX: track 30.4 -> 31.4 mm
- net TX1: track 8.45 -> 7.40 mm
- net +9V: track 27.2 -> 28.2 mm
- net RX0: track 19.6 -> 19.0 mm
- net TX: track 31.9 -> 31.4 mm
- net GND: vias 64 -> 53
- net (no net): vias 0 -> 3
Other:
- board text added: "espSFD"
