File: hardware/pcb/espSFD/espSFD.kicad_sch (KiCad schematic)
At the start: 9 parts, among them J1 Conn_01x06_Socket, J2 Conn_02x10_Odd_Even, Q1 IRLU3110Z, U1 WeMos_D1_mini, U2 TSR_1-2415

Commit message: xhd
Parts:
- H1, H2: footprint MountingHole:MountingHole_3.2mm_M3_Pad -> MountingHole:MountingHole_3.2mm_M3_DIN965_Pad
Changed lines of the file:
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@@
       (effects (font (size 1.27 1.27)) (justify left) hide)
     )
-    (property "Footprint" "MountingHole:MountingHole_3.2mm_M3_Pad" (at 107.95 114.3 0)
+    (property "Footprint" "MountingHole:MountingHole_3.2mm_M3_DIN965_Pad" (at 107.95 114.3 0)
       (effects (font (size 1.27 1.27)) hide)
     )
@@
       (effects (font (size 1.27 1.27)) (justify left) hide)
     )
-    (property "Footprint" "MountingHole:MountingHole_3.2mm_M3_Pad" (at 100.33 114.3 0)
+    (property "Footprint" "MountingHole:MountingHole_3.2mm_M3_DIN965_Pad" (at 100.33 114.3 0)
       (effects (font (size 1.27 1.27)) hide)
     )

Commit message: es dghdgfj fcgj
Parts:
- added JP1, JP2: SolderJumper_3_Open, Library:SolderJumper-3_P1.3mm_Open_Pad1.0x1.5mm no silk, symbol Jumper:SolderJumper_3_Open
Connections:
- net RX: now also J2.19 (Pin_19), JP1.2 (C); no longer J2.17 (Pin_17), U1.11 (D4)
- net TX: now also J2.17 (Pin_17), JP2.2 (C); no longer J2.19 (Pin_19), U1.12 (D3)
- net RX0: now reaches U1.15 (RX)
- net RX0: now also JP1.1 (A)
- net TX0: now reaches U1.16 (TX)
- net TX0: now also JP2.1 (A)
- new net RX1: JP1.3 (B), U1.11 (D4)
- new net TX1: JP2.3 (B), U1.12 (D3)
- no-connect marks 11 -> 9
Changed lines of the file:
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@@
   (junction (at 102.87 50.8) (diameter 0) (color 0 0 0 0)
   )
-  (no_connect (at 200.66 100.33))
   (no_connect (at 220.98 113.03))
   (no_connect (at 213.36 82.55))
@@
   (no_connect (at 220.98 90.17))
   (no_connect (at 220.98 107.95))
-  (no_connect (at 200.66 102.87))
   (no_connect (at 220.98 95.25))
   (no_connect (at 220.98 97.79))
@@
     (stroke (width 0) (type default))
   )
-  (global_label "TX" (shape input) (at 115.57 48.26 0) (fields_autoplaced)
-    (effects (font (size 1.27 1.27)) (justify left))
-    (property "Intersheetrefs" "${INTERSHEET_REFS}" (at 120.7323 48.26 0)
+  (global_label "TX" (shape input) (at 115.57 50.8 0) (fields_autoplaced)
+    (effects (font (size 1.27 1.27)) (justify left))
+    (property "Intersheetrefs" "${INTERSHEET_REFS}" (at 120.7323 50.8 0)
       (effects (font (size 1.27 1.27)) (justify left) hide)
     )
@@
     )
   )
-  (global_label "RX" (shape input) (at 115.57 50.8 0) (fields_autoplaced)
-    (effects (font (size 1.27 1.27)) (justify left))
-    (property "Intersheetrefs" "${INTERSHEET_REFS}" (at 121.0347 50.8 0)
-      (effects (font (size 1.27 1.27)) (justify left) hide)
-    )
-  )
-  (global_label "TX" (shape input) (at 220.98 100.33 0) (fields_autoplaced)
-    (effects (font (size 1.27 1.27)) (justify left))
-    (property "Intersheetrefs" "${INTERSHEET_REFS}" (at 226.1423 100.33 0)
+  (global_label "RX" (shape input) (at 115.57 48.26 0) (fields_autoplaced)
+    (effects (font (size 1.27 1.27)) (justify left))
+    (property "Intersheetrefs" "${INTERSHEET_REFS}" (at 121.0347 48.26 0)
+      (effects (font (size 1.27 1.27)) (justify left) hide)
+    )
+  )
+  (global_label "RX1" (shape input) (at 153.67 90.17 180) (fields_autoplaced)
+    (effects (font (size 1.27 1.27)) (justify right))
+    (property "Intersheetrefs" "${INTERSHEET_REFS}" (at 146.9958 90.17 0)
+      (effects (font (size 1.27 1.27)) (justify right) hide)
+    )
+  )
+  (global_label "TX1" (shape input) (at 153.67 106.68 180) (fields_autoplaced)
+    (effects (font (size 1.27 1.27)) (justify right))
+    (property "Intersheetrefs" "${INTERSHEET_REFS}" (at 147.2982 106.68 0)
+      (effects (font (size 1.27 1.27)) (justify right) hide)
+    )
+  )
+  (global_label "RX0" (shape input) (at 163.83 90.17 0) (fields_autoplaced)
+    (effects (font (size 1.27 1.27)) (justify left))
+    (property "Intersheetrefs" "${INTERSHEET_REFS}" (at 170.5042 90.17 0)
+      (effects (font (size 1.27 1.27)) (justify left) hide)
+    )
+  )
+  (global_label "TX" (shape input) (at 158.75 110.49 270) (fields_autoplaced)
+    (effects (font (size 1.27 1.27)) (justify right))
+    (property "Intersheetrefs" "${INTERSHEET_REFS}" (at 158.75 115.6523 90)
+      (effects (font (size 1.27 1.27)) (justify right) hide)
+    )
+  )
+  (global_label "TX1" (shape input) (at 220.98 100.33 0) (fields_autoplaced)
+    (effects (font (size 1.27 1.27)) (justify left))
+    (property "Intersheetrefs" "${INTERSHEET_REFS}" (at 227.3518 100.33 0)
       (effects (font (size 1.27 1.27)) (justify left) hide)
     )
@@
     )
   )
+  (global_label "RX0" (shape input) (at 200.66 100.33 180) (fields_autoplaced)
+    (effects (font (size 1.27 1.27)) (justify right))
+    (property "Intersheetrefs" "${INTERSHEET_REFS}" (at 193.9858 100.33 0)
+      (effects (font (size 1.27 1.27)) (justify right) hide)
+    )
+  )
+  (global_label "TX0" (shape input) (at 163.83 106.68 0) (fields_autoplaced)
+    (effects (font (size 1.27 1.27)) (justify left))
+    (property "Intersheetrefs" "${INTERSHEET_REFS}" (at 170.2018 106.68 0)
+      (effects (font (size 1.27 1.27)) (justify left) hide)
+    )
+  )
   (global_label "Motor N" (shape input) (at 115.57 71.12 0) (fields_autoplaced)
     (effects (font (size 1.27 1.27)) (justify left))
@@
     )
   )
+  (global_label "TX0" (shape input) (at 200.66 102.87 180) (fields_autoplaced)
+    (effects (font (size 1.27 1.27)) (justify right))
+    (property "Intersheetrefs" "${INTERSHEET_REFS}" (at 194.2882 102.87 0)
+      (effects (font (size 1.27 1.27)) (justify right) hide)
+    )
+  )
   (global_label "En Motor" (shape input) (at 237.49 86.36 90) (fields_autoplaced)
     (effects (font (size 1.27 1.27)) (justify left))
@@
     )
   )
-  (global_label "RX" (shape input) (at 220.98 102.87 0) (fields_autoplaced)
-    (effects (font (size 1.27 1.27)) (justify left))
-    (property "Intersheetrefs" "${INTERSHEET_REFS}" (at 226.4447 102.87 0)
+  (global_label "RX" (shape input) (at 158.75 93.98 270) (fields_autoplaced)
+    (effects (font (size 1.27 1.27)) (justify right))
+    (property "Intersheetrefs" "${INTERSHEET_REFS}" (at 158.75 99.4447 90)
+      (effects (font (size 1.27 1.27)) (justify right) hide)
+    )
+  )
+  (global_label "RX1" (shape input) (at 220.98 102.87 0) (fields_autoplaced)
+    (effects (font (size 1.27 1.27)) (justify left))
+    (property "Intersheetrefs" "${INTERSHEET_REFS}" (at 227.6542 102.87 0)
       (effects (font (size 1.27 1.27)) (justify left) hide)
     )
@@
         (path "/b4f72b7f-c57f-4eed-9610-6133338117bb"
           (reference "#PWR09") (unit 1)
+        )
+      )
+    )
+  )
+  (symbol (lib_id "Jumper:SolderJumper_3_Open") (at 158.75 106.68 0) (mirror y) (unit 1)
+    (in_bom yes) (on_board yes) (dnp no)
+    (property "Reference" "JP2" (at 158.75 100.33 0)
+      (effects (font (size 1.27 1.27)))
+    )
+    (property "Value" "SolderJumper_3_Open" (at 158.75 102.87 0)
+      (effects (font (size 1.27 1.27)))
+    )
+    (property "Footprint" "Library:SolderJumper-3_P1.3mm_Open_Pad1.0x1.5mm no silk" (at 158.75 106.68 0)
+      (effects (font (size 1.27 1.27)) hide)
+    )
+    (property "Datasheet" "~" (at 158.75 106.68 0)
+      (effects (font (size 1.27 1.27)) hide)
+    )
+    (pin "3")
+    (pin "2")
+    (pin "1")
+    (instances
+      (project "espSFD"
+        (path "/b4f72b7f-c57f-4eed-9610-6133338117bb"
+          (reference "JP2") (unit 1)
         )
       )
@@
         )
       )
+    )
+  )
+  (symbol (lib_id "Jumper:SolderJumper_3_Open") (at 158.75 90.17 0) (mirror y) (unit 1)
+    (in_bom yes) (on_board yes) (dnp no)
+    (property "Reference" "JP1" (at 158.75 83.82 0)
+      (effects (font (size 1.27 1.27)))
+    )
+    (property "Value" "SolderJumper_3_Open" (at 158.75 86.36 0)
+      (effects (font (size 1.27 1.27)))
+    )
+    (property "Footprint" "Library:SolderJumper-3_P1.3mm_Open_Pad1.0x1.5mm no silk" (at 158.75 90.17 0)
+      (effects (font (size 1.27 1.27)) hide)
+    )
+    (property "Datasheet" "~" (at 158.75 90.17 0)
+      (effects (font (size 1.27 1.27)) hide)
+    )
+    (pin "3")
+    (pin "2")
+    (pin "1")
+    (instances
+      (project "espSFD"
+        (path "/b4f72b7f-c57f-4eed-9610-6133338117bb"
+          (reference "JP1") (unit 1)
+        )
+      )

Commit message: vcb
Signed-off-by: Christian Backus <chrissileinus@googlemail.com>
Parts:
- removed H1, H2: MountingHole_Pad, MountingHole:MountingHole_3.2mm_M3_DIN965_Pad, symbol Mechanical:MountingHole_Pad
- added DRA1, DRA2: DIN_Rail_Adapter, Library:DINRailAdapter_3xM3_PhoenixContact_1201578, symbol Mechanical:DIN_Rail_Adapter
- U1: value WeMos_D1_mini -> WeMos_D1_mini_esp32
Changed lines of the file:
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@@
+    )
+  )
+  (symbol (lib_id "Mechanical:DIN_Rail_Adapter") (at 55.88 146.05 0) (unit 1)
+    (in_bom yes) (on_board yes) (dnp no) (fields_autoplaced)
+    (property "Reference" "DRA1" (at 55.88 138.43 0)
+      (effects (font (size 1.27 1.27)))
+    )
+    (property "Value" "DIN_Rail_Adapter" (at 55.88 140.97 0)
+      (effects (font (size 1.27 1.27)))
+    )
+    (property "Footprint" "Library:DINRailAdapter_3xM3_PhoenixContact_1201578" (at 55.88 151.13 0)
+      (effects (font (size 1.27 1.27)) hide)
+    )
+    (property "Datasheet" "~" (at 55.88 142.24 0)
+      (effects (font (size 1.27 1.27)) hide)
+    )
+    (instances
+      (project "espSFD"
+        (path "/b4f72b7f-c57f-4eed-9610-6133338117bb"
+          (reference "DRA1") (unit 1)
+        )
+      )
     )
   )
@@
       (effects (font (size 1.27 1.27)) (justify left))
     )
-    (property "Value" "WeMos_D1_mini" (at 213.0141 125.73 0)
+    (property "Value" "WeMos_D1_mini_esp32" (at 213.0141 125.73 0)
       (effects (font (size 1.27 1.27)) (justify left))
     )
@@
     )
   )
-  (symbol (lib_id "Mechanical:MountingHole_Pad") (at 107.95 114.3 0) (unit 1)
-    (in_bom yes) (on_board yes) (dnp no) (fields_autoplaced)
-    (property "Reference" "H1" (at 110.49 111.76 0)
-      (effects (font (size 1.27 1.27)) (justify left))
-    )
-    (property "Value" "MountingHole_Pad" (at 110.49 114.3 0)
-      (effects (font (size 1.27 1.27)) (justify left) hide)
-    )
-    (property "Footprint" "MountingHole:MountingHole_3.2mm_M3_DIN965_Pad" (at 107.95 114.3 0)
-      (effects (font (size 1.27 1.27)) hide)
-    )
-    (property "Datasheet" "~" (at 107.95 114.3 0)
-      (effects (font (size 1.27 1.27)) hide)
-    )
-    (pin "1")
-    (instances
-      (project "espSFD"
-        (path "/b4f72b7f-c57f-4eed-9610-6133338117bb"
-          (reference "H1") (unit 1)
-        )
-      )
-    )
-  )
   (symbol (lib_id "PCM_Transistor_MOSFET_AKL:IRLU3110Z") (at 234.95 91.44 0) (unit 1)
     (in_bom yes) (on_board yes) (dnp no) (fields_autoplaced)
@@
     )
   )
+  (symbol (lib_id "Mechanical:DIN_Rail_Adapter") (at 52.07 166.37 0) (unit 1)
+    (in_bom yes) (on_board yes) (dnp no) (fields_autoplaced)
+    (property "Reference" "DRA2" (at 52.07 158.75 0)
+      (effects (font (size 1.27 1.27)))
+    )
+    (property "Value" "DIN_Rail_Adapter" (at 52.07 161.29 0)
+      (effects (font (size 1.27 1.27)))
+    )
+    (property "Footprint" "Library:DINRailAdapter_3xM3_PhoenixContact_1201578" (at 52.07 171.45 0)
+      (effects (font (size 1.27 1.27)) hide)
+    )
+    (property "Datasheet" "~" (at 52.07 162.56 0)
+      (effects (font (size 1.27 1.27)) hide)
+    )
+    (instances
+      (project "espSFD"
+        (path "/b4f72b7f-c57f-4eed-9610-6133338117bb"
+          (reference "DRA2") (unit 1)
+        )
+      )
+    )
+  )
   (symbol (lib_id "power:GND") (at 237.49 96.52 0) (unit 1)
     (in_bom yes) (on_board yes) (dnp no) (fields_autoplaced)
@@
         (path "/b4f72b7f-c57f-4eed-9610-6133338117bb"
           (reference "#PWR013") (unit 1)
-        )
-      )
-    )
-  )
-  (symbol (lib_id "power:GND") (at 107.95 116.84 0) (unit 1)
-    (in_bom yes) (on_board yes) (dnp no) (fields_autoplaced)
-    (property "Reference" "#PWR012" (at 107.95 123.19 0)
-      (effects (font (size 1.27 1.27)) hide)
-    )
-    (property "Value" "GND" (at 107.95 121.92 0)
-      (effects (font (size 1.27 1.27)))
-    )
-    (property "Footprint" "" (at 107.95 116.84 0)
-      (effects (font (size 1.27 1.27)) hide)
-    )
-    (property "Datasheet" "" (at 107.95 116.84 0)
-      (effects (font (size 1.27 1.27)) hide)
-    )
-    (pin "1")
-    (instances
-      (project "espSFD"
-        (path "/b4f72b7f-c57f-4eed-9610-6133338117bb"
-          (reference "#PWR012") (unit 1)
         )
       )
@@
         (path "/b4f72b7f-c57f-4eed-9610-6133338117bb"
           (reference "#PWR01") (unit 1)
-        )
-      )
-    )
-  )
-  (symbol (lib_id "Mechanical:MountingHole_Pad") (at 100.33 114.3 0) (unit 1)
-    (in_bom yes) (on_board yes) (dnp no) (fields_autoplaced)
-    (property "Reference" "H2" (at 102.87 111.76 0)
-      (effects (font (size 1.27 1.27)) (justify left))
-    )
-    (property "Value" "MountingHole_Pad" (at 102.87 114.3 0)
-      (effects (font (size 1.27 1.27)) (justify left) hide)
-    )
-    (property "Footprint" "MountingHole:MountingHole_3.2mm_M3_DIN965_Pad" (at 100.33 114.3 0)
-      (effects (font (size 1.27 1.27)) hide)
-    )
-    (property "Datasheet" "~" (at 100.33 114.3 0)
-      (effects (font (size 1.27 1.27)) hide)
-    )
-    (pin "1")
-    (instances
-      (project "espSFD"
-        (path "/b4f72b7f-c57f-4eed-9610-6133338117bb"
-          (reference "H2") (unit 1)
         )
       )
@@
         )
       )
-    )
-  )
-  (symbol (lib_id "power:GND") (at 100.33 116.84 0) (unit 1)
-    (in_bom yes) (on_board yes) (dnp no) (fields_autoplaced)
-    (property "Reference" "#PWR011" (at 100.33 123.19 0)
-      (effects (font (size 1.27 1.27)) hide)
-    )
-    (property "Value" "GND" (at 100.33 121.92 0)
-      (effects (font (size 1.27 1.27)))
-    )
-    (property "Footprint" "" (at 100.33 116.84 0)
-      (effects (font (size 1.27 1.27)) hide)
-    )
-    (property "Datasheet" "" (at 100.33 116.84 0)
-      (effects (font (size 1.27 1.27)) hide)
-    )
-    (pin "1")
-    (instances
-      (project "espSFD"
-        (path "/b4f72b7f-c57f-4eed-9610-6133338117bb"
-          (reference "#PWR011") (unit 1)
-        )
-      )
