File: hardware/pcb/espSFDmains/espSFDmains.kicad_pcb (KiCad board)
At the start: 2 copper layers, 69 x 35 mm, 11 parts, among them J1 Conn_01x06_Socket, J2 Conn_02x10_Odd_Even, Q1 IRLU3110Z, U1 WeMos_D1_mini_esp32, U2 TSR_1-2415

Commit message: add espSFDmains
Parts:
- added F1: 1A, Fuse:Fuseholder_TR5_Littelfuse_No560_No460, F.Cu at (105.4, 135.9)
- added J3: Conn_01x02_Socket, Connector_Phoenix_MSTB:PhoenixContact_MSTBA_2,5_2-G-5,08_1x02_P5.08mm_Horizontal, F.Cu at (100.3, 125.7)
- added PS2: TPP-15-109-D, Converter_ACDC:Converter_ACDC_TRACO_TPP-15-1xx-D_THT, F.Cu at (88.4, 129.6)
Routing:
- net +9V: track 28.2 -> 105.8 mm
- net NEUT: track 0.00 -> 17.6 mm
- net LINE: track 0.00 -> 13.8 mm
- net Net-(PS2-AC/L): track 0.00 -> 12.2 mm
- net GND: vias 53 -> 51
Other:
- board size 69 x 35 mm -> 69 x 65 mm
- board text added: "230~"
- board text added: "L"
- board text added: "N"

Commit message: ghjfgj
Parts:
- removed Q1: IRLU3110Z, PCM_Package_TO_SOT_THT_AKL:TO-251-3_Vertical_GDS
- added 5V1: LED, LED_THT:LED_D3.0mm, F.Cu at (137.5, 107.6)
- added 9V1: LED, LED_THT:LED_D3.0mm, F.Cu at (141.9, 107.6)
- added F2: 6A, Fuse:Fuseholder_TR5_Littelfuse_No560_No460, F.Cu at (140.7, 142.6)
- added J4: Mains Motor, Connector_Phoenix_MSTB:PhoenixContact_MSTBA_2,5_2-G-5,08_1x02_P5.08mm_Horizontal, F.Cu at (137.5, 122.2)
- added K1: SKB10420, KiCad:SKB10420, F.Cu at (121.6, 141.3)
- added Q2: BS170, PCM_Package_TO_SOT_THT_AKL:TO-92_Inline_Wide_DGS, F.Cu at (111.4, 102.5)
- added R3: 180R, Resistor_THT:R_Axial_DIN0204_L3.6mm_D1.6mm_P7.62mm_Horizontal, F.Cu at (134.3, 107.6)
- added R4: 180R, Resistor_THT:R_Axial_DIN0204_L3.6mm_D1.6mm_P7.62mm_Horizontal, F.Cu at (134.3, 105.1)
- added R5: 4K7, Resistor_THT:R_Axial_DIN0204_L3.6mm_D1.6mm_P7.62mm_Horizontal, F.Cu at (102.5, 86.7)
- added R6: 4K7, Resistor_THT:R_Axial_DIN0204_L3.6mm_D1.6mm_P7.62mm_Horizontal, F.Cu at (105.1, 86.7)
- J1: footprint Connector_Phoenix_MSTB:PhoenixContact_MSTBA_2,5_6-G-5,08_1x06_P5.08mm_Horizontal -> Connector_Phoenix_MC:PhoenixContact_MC_1,5_6-G-3.81_1x06_P3.81mm_Horizontal
- J3: value Conn_01x02_Socket -> Mains
- R2: value 2K2 -> 180K
- U2: value TSR_1-2415 -> TSR_1-2450
- moved DRA2 91.4 mm to (126.0, 154.0), turned to 0 degrees
- moved DRA1 63.9 mm to (126.0, 75.2), turned to 0 degrees
- moved J1 39.5 mm to (139.4, 100.6)
- moved J3 38.6 mm to (137.5, 136.2)
- moved U1 34.5 mm to (84.8, 79.0)
- moved J2 31.7 mm to (122.2, 75.2)
- moved U2 31.6 mm to (112.7, 90.5)
- moved JP2 31.4 mm to (96.2, 89.2)
- moved JP1 31.4 mm to (96.2, 91.8)
- moved R2 30.5 mm to (100.0, 102.5)
- moved R1 30.5 mm to (92.4, 100.0)
- moved F1 26.0 mm to (130.5, 142.6), turned to -90 degrees
- moved PS2 18.0 mm to (94.9, 146.4), turned to 90 degrees
Connections:
- J1 pad 3: +9V -> SDA
- J1 pad 4: En Motor -> SCL
- U1 pad 13: unconnected-(U1-SDA/D2-Pad13) -> SDA
- U1 pad 14: unconnected-(U1-SCL/D1-Pad14) -> SCL
Routing:
- net NEUT: track 17.6 -> 68.7 mm
- net SCL: track 0.00 -> 40.0 mm
- net En Motor: track 37.9 -> 0.00 mm
- net SDA: track 0.00 -> 36.9 mm
- net Net-(PS2-AC/L): track 12.2 -> 44.8 mm
- net Net-(K1-~_1): track 0.00 -> 21.7 mm
- net +5V: track 9.20 -> 29.7 mm
- net 230V Motor: track 0.00 -> 19.6 mm
- net Net-(K1--): track 0.00 -> 15.6 mm
- net Net-(9V1-A): track 0.00 -> 8.67 mm
- net +9V: track 105.8 -> 97.1 mm
- net Motor N: track 22.1 -> 30.4 mm
- net Net-(U1-D0): track 12.7 -> 19.0 mm
- net Motor L: track 23.8 -> 29.8 mm
- net LINE: track 13.8 -> 19.1 mm
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- added copper zone on F.Cu, net Motor L
- added copper zone on F.Cu, net Motor N
- removed copper zone on B.Cu, net Motor L
- removed copper zone on B.Cu, net Motor N
Other:
- board size 69 x 65 mm -> 64 x 88.9 mm
- board text added: "1A"
- board text added: "42V AC"
- board text added: "5V"
- board text added: "6A"
- board text added: "9V"
- board text added: "9V DC"
- board text added: "I²C Bus"
- board text added: "I²C PullUp"
- board text added: "Mains 230V AC"
- board text added: "Motor"
- board text added: "Motor 230V AC"
- board text added: "SCL"
- board text added: "SDL"
- board text added: "SFD Bus"
- board text removed: "+9V"
- board text removed: "230~"
- board text removed: "Bus"
- board text removed: "En"
- board text removed: "RX0"
- board text removed: "RX1"
- board text removed: "TX0"
- board text removed: "TX1"
- board text removed: "~42V"

Commit message: fdshd f
Parts:
- added PS1: TMLM20105, Converter_ACDC:Converter_ACDC_TRACO_TMLM-10-20_THT, F.Cu at (96.7, 109.8)
- moved PS2 1.53 mm to (94.9, 144.8)
Routing:
- net NEUT: track 68.7 -> 78.8 mm
- net Net-(PS2-AC/L): track 44.8 -> 52.5 mm
- net +9V: track 97.1 -> 98.7 mm
Other:
- outline, holes or cut-outs redrawn

Commit message: etw erzt
Parts:
- removed K1: SKB10420, KiCad:SKB10420
- removed PS1: TMLM20105, Converter_ACDC:Converter_ACDC_TRACO_TMLM-10-20_THT
- removed Q2: BS170, PCM_Package_TO_SOT_THT_AKL:TO-92_Inline_Wide_DGS
- removed R2: 180K, Resistor_THT:R_Axial_DIN0204_L3.6mm_D1.6mm_P7.62mm_Horizontal
- added S1: CPC40055ST, lib:CPC40055ST, F.Cu at (103.8, 147.4)
- moved 9V1 53.3 mm to (88.6, 107.0), turned to 0 degrees
- moved 5V1 49.2 mm to (88.6, 101.9), turned to 0 degrees
- moved R3 40.7 mm to (93.7, 105.7), turned to 0 degrees
- moved R4 40.7 mm to (93.7, 103.2), turned to 0 degrees
- moved PS2 30.9 mm to (123.5, 133.0), turned to 180 degrees
- moved U1 15.9 mm to (86.0, 94.9), turned to 90 degrees
- moved R6 15.7 mm to (93.7, 75.9)
- moved R5 15.7 mm to (91.1, 75.9)
- moved U2 14.5 mm to (116.5, 104.5), turned to 180 degrees
- moved JP1 12.3 mm to (98.7, 79.7), turned to 90 degrees
- moved F1 12.1 mm to (142.6, 142.6)
- moved JP2 9.52 mm to (96.2, 79.7), turned to 90 degrees
- moved F2 8.25 mm to (132.4, 142.6)
- moved J2 6.63 mm to (124.1, 81.6)
- moved R1 1.42 mm to (93.7, 100.6)
Routing:
- net NEUT: track 78.8 -> 34.6 mm
- net Net-(S1-+LED): track 17.6 -> 49.1 mm
- net +5V: track 29.7 -> 59.7 mm, vias 0 -> 1
- net Net-(PS2-AC/L): track 52.5 -> 22.8 mm
- net 230V Motor: track 19.6 -> 42.8 mm
- net SDA: track 36.9 -> 58.4 mm
- net SCL: track 40.0 -> 59.2 mm
- net GND: track 0.00 -> 17.8 mm, vias 0 -> 1
- net Net-(K1--): track 15.6 -> 0.00 mm
- net Net-(U1-D0): track 19.0 -> 6.77 mm
- net RX: track 29.6 -> 39.3 mm
- net +9V: track 98.7 -> 89.5 mm
- net Net-(S1-AC_LOAD1): track 21.7 -> 13.3 mm
- net TX0: track 22.2 -> 15.3 mm, vias 0 -> 1
- net TX: track 31.6 -> 38.3 mm
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- added copper zone on B.Cu, net Motor L
- added copper zone on B.Cu, net Motor N
Other:
- board size 64 x 88.9 mm -> 62.9 x 88.9 mm
- board text removed: "1A"
- board text removed: "6A"
- board text removed: "Motor 230V AC"

Commit message: gfjhdfjh
Parts:
- removed 5V1, 9V1: LED, LED_THT:LED_D3.0mm
- removed R3, R4: 180R, Resistor_THT:R_Axial_DIN0204_L3.6mm_D1.6mm_P7.62mm_Horizontal
- added C1: 100µ/25V, Capacitor_THT:CP_Radial_D5.0mm_P2.00mm, F.Cu at (121.6, 83.8)
- added D1: 1N4148, Diode_THT:D_DO-35_SOD27_P7.62mm_Horizontal, F.Cu at (124.1, 96.8)
- added R2: 180R, Resistor_THT:R_Axial_DIN0204_L3.6mm_D1.6mm_P7.62mm_Horizontal, F.Cu at (121.6, 96.8)
- added R7: 180R, Resistor_THT:R_Axial_DIN0204_L3.6mm_D1.6mm_P7.62mm_Horizontal, F.Cu at (107.6, 101.9)
- added U3: SFH617A-1, Package_DIP:DIP-4_W7.62mm, F.Cu at (119.1, 89.2)
- moved R1 40.7 mm to (92.4, 141.3)
- moved JP1 14.8 mm to (105.1, 93.0)
- moved JP2 14.8 mm to (102.5, 93.0)
- moved R6 12.5 mm to (100.0, 86.7), turned to 0 degrees
- moved R5 12.1 mm to (100.0, 84.1), turned to 0 degrees
- moved U1 10.3 mm to (89.8, 104.5)
- moved U2 6.84 mm to (122.9, 107.0), turned to 90 degrees
- moved PS2 6.35 mm to (127.3, 127.9)
- moved J2 5.08 mm to (129.2, 81.6)
- moved S1 3.81 mm to (107.6, 147.4)
- moved F2 0.64 mm to (131.8, 142.6)
Connections:
- net +5V renamed VCC
- net +9V renamed VDD
- net GND renamed VSS
- U1 pad 4: unconnected-(U1-SCK/D5-Pad4) -> Det. Motor Supply
Routing:
- net Net-(S1-+LED): track 49.1 -> 6.35 mm
- net Net-(U1-D0): track 6.77 -> 40.8 mm
- net VCC: track 59.7 -> 31.1 mm, vias 1 -> 0
- net Det. Motor Supply: track 0.00 -> 25.1 mm, vias 0 -> 2
- net VDD: track 89.5 -> 70.8 mm
- net VSS: track 17.8 -> 0.00 mm, vias 1 -> 0
- net SDA: track 58.4 -> 48.1 mm, vias 0 -> 4
- net SCL: track 59.2 -> 49.2 mm, vias 0 -> 4
- net TX: track 38.3 -> 32.2 mm, vias 0 -> 3
- net RX: track 39.3 -> 33.7 mm, vias 0 -> 3
- net RX0: track 17.5 -> 22.7 mm, vias 1 -> 2
- net Motor N: track 27.9 -> 22.9 mm
- net RX1: track 6.32 -> 11.1 mm
- net TX1: track 6.32 -> 11.1 mm
- net Net-(S1-AC_LOAD1): track 13.3 -> 8.88 mm
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- removed copper zone on B.Cu, net Motor L
- removed copper zone on B.Cu, net Motor N
Other:
- board size 62.9 x 88.9 mm -> 59.1 x 88.9 mm
- board text added: "0V DC"
- board text added: "6V DC"
- board text added: "Mains In"
- board text removed: "5V"
- board text removed: "9V"
- board text removed: "9V DC"
- board text removed: "GND"
- board text removed: "Mains 230V AC"

Commit message: bsfnbdfnb
Parts:
- removed C1: 100µ/25V, Capacitor_THT:CP_Radial_D5.0mm_P2.00mm
- removed D1: 1N4148, Diode_THT:D_DO-35_SOD27_P7.62mm_Horizontal
- removed R2, R7: 180R, Resistor_THT:R_Axial_DIN0204_L3.6mm_D1.6mm_P7.62mm_Horizontal
- removed R5, R6: 4K7, Resistor_THT:R_Axial_DIN0204_L3.6mm_D1.6mm_P7.62mm_Horizontal
- removed U3: SFH617A-1, Package_DIP:DIP-4_W7.62mm
- added J5: Motor, Connector_Phoenix_MC:PhoenixContact_MC_1,5_2-G-3.81_1x02_P3.81mm_Horizontal, F.Cu at (143.2, 111.4)
- J1: value Conn_01x06_Socket -> VDD; footprint Connector_Phoenix_MC:PhoenixContact_MC_1,5_6-G-3.81_1x06_P3.81mm_Horizontal -> Connector_Phoenix_MC:PhoenixContact_MC_1,5_2-G-3.81_1x02_P3.81mm_Horizontal
- J3, J4: footprint Connector_Phoenix_MSTB:PhoenixContact_MSTBA_2,5_2-G-5,08_1x02_P5.08mm_Horizontal -> Connector_Phoenix_MC:PhoenixContact_MC_1,5_2-G-3.81_1x02_P3.81mm_Horizontal
- R1: value 180R -> 100R
- moved R1 34.7 mm to (97.5, 107.0), turned to 180 degrees
- moved U2 27.9 mm to (143.2, 87.9)
- moved J2 23.0 mm to (131.8, 104.5), turned to 180 degrees
- moved F2 17.9 mm to (138.7, 126.0), turned to 180 degrees
- moved J4 8.08 mm to (143.2, 127.9)
- moved J3 7.24 mm to (143.2, 140.6)
- moved JP1 6.25 mm to (102.5, 87.3)
- moved JP2 6.25 mm to (100.0, 87.3)
- moved DRA2 5.99 mm to (129.2, 148.9)
- moved F1 5.39 mm to (138.7, 138.7), turned to 180 degrees
- moved S1 5.08 mm to (107.6, 142.4)
- moved J1 4.26 mm to (143.2, 98.7)
- moved DRA1 3.17 mm to (129.2, 75.2)
Connections:
- net Net-(U1-D0) renamed En Motor
- F2 pad 1: LINE -> 230V Motor
- F2 pad 2: Net-(S1-AC_LOAD1) -> Net-(S1-AC_LOAD2)
- S1 pad 1: Net-(S1-AC_LOAD1) -> LINE
- S1 pad 2: 230V Motor -> Net-(S1-AC_LOAD2)
- U1 pad 13: SDA -> unconnected-(U1-SDA/D2-Pad13)
- U1 pad 14: SCL -> unconnected-(U1-SCL/D1-Pad14)
- U1 pad 4: Det. Motor Supply -> unconnected-(U1-SCK/D5-Pad4)
Routing:
- net SCL: track 49.2 -> 0.00 mm, vias 4 -> 0
- net SDA: track 48.1 -> 0.00 mm, vias 4 -> 0
- net Net-(S1-+LED): track 6.35 -> 46.6 mm
- net 230V Motor: track 42.7 -> 5.23 mm
- net En Motor: track 40.8 -> 3.59 mm
- net Net-(S1-AC_LOAD2): track 0.00 -> 32.2 mm
- net Det. Motor Supply: track 25.1 -> 0.00 mm, vias 2 -> 0
- net VDD: track 70.8 -> 86.7 mm
- net Net-(PS2-AC/L): track 21.1 -> 8.50 mm
- net Net-(S1-AC_LOAD1): track 8.88 -> 0.00 mm
- net Motor N: track 22.9 -> 29.8 mm
- net RX1: track 11.1 -> 4.41 mm
- net TX1: track 11.1 -> 4.41 mm
- net VCC: track 31.1 -> 37.7 mm
- net LINE: track 17.2 -> 22.7 mm
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Other:
- board size 59.1 x 88.9 mm -> 62.2 x 83.8 mm
- board text added: "1A"
- board text added: "6A"
- board text added: "9V DC"
- board text added: "Mains"
- board text added: "chrissileinus"
- board text removed: "6V DC"
- board text removed: "I²C Bus"
- board text removed: "I²C PullUp"
- board text removed: "Mains In"
- board text removed: "SCL"
- board text removed: "SDL"

Commit message: hfdghd
Parts:
- moved R1 2.54 mm to (97.5, 109.5)
Routing:
- net Net-(S1-+LED): track 46.6 -> 44.0 mm
- net En Motor: track 3.59 -> 6.13 mm
Changed lines of the file:
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@@
 		)
 		(property "Value" "6A"
-			(at 6.985 -3.81 270)
+			(at 6.985 -3.81 -90)
 			(layer "F.Fab")
 			(effects
@@
 		(tags "DCDC-Converter TRACO TSR-1")
 		(property "Reference" "U2"
-			(at -1.5 -6.71 270)
+			(at -1.5 -6.71 -90)
 			(layer "F.SilkS")
 			(hide yes)
@@
 		)
 		(property "Value" "TSR_1-2450"
-			(at -2.58 9.6 270)
+			(at -2.58 9.6 -90)
 			(layer "F.Fab")
 			(hide yes)
@@
 		)
 		(fp_text user "${REFERENCE}"
-			(at 3 -3 270)
+			(at 3 -3 -90)
 			(layer "F.Fab")
 			(effects
@@
 		)
 		(property "Value" "1A"
-			(at 6.985 -3.81 270)
+			(at 6.985 -3.81 -90)
 			(layer "F.Fab")
 			(effects
@@
 		)
 		(fp_text user "${REFERENCE}"
-			(at 1.27 11.43 270)
+			(at 1.27 11.43 -90)
 			(layer "F.Fab")
 			(effects
@@
 	(footprint "Resistor_THT:R_Axial_DIN0204_L3.6mm_D1.6mm_P7.62mm_Horizontal"
 		(layer "F.Cu")
-		(at 97.47 106.99 180)
+		(at 97.47 109.53 180)
 		(descr "Resistor, Axial_DIN0204 series, Axial, Horizontal, pin pitch=7.62mm, 0.167W, length*diameter=3.6*1.6mm^2, http://cdn-reichelt.de/documents/datenblatt/B400/1_4W%23YAG.pdf")
 		(tags "Resistor Axial_DIN0204 series Axial Horizontal pin pitch 7.62mm 0.167W length 3.6mm diameter 1.6mm")
@@
 	)
 	(segment
+		(start 97.47 109.53)
+		(end 97.47 106.99)
+		(width 0.25)
+		(layer "F.Cu")
+		(net 11)
+	)
+	(segment
 		(start 97.47 106.99)
 		(end 94.93 104.45)
@@
 	)
 	(segment
-		(start 89.85 106.99)
+		(start 89.85 109.53)
 		(end 89.85 141.28)
 		(width 0.25)

Commit message: PCB V1.2
Parts:
- removed U1: WeMos_D1_mini_esp32, Module:WEMOS_D1_mini_light
- added C1: 15µF/50V, Capacitor_Tantalum_SMD:CP_EIA-7343-43_Kemet-X, B.Cu at (100.6, 143.8)
- added C2: 10nF/50V, Capacitor_SMD:C_0805_2012Metric, B.Cu at (97.5, 133.7)
- added C3: 68µF/16V, Capacitor_Tantalum_SMD:CP_EIA-7343-43_Kemet-X, B.Cu at (100.0, 127.3)
- added C4: 0.1uF/275Vac, Capacitor_THT:C_Rect_L16.5mm_W5.0mm_P15.00mm_MKT, F.Cu at (46.8, 117.2)
- added D1: SS14, Diode_SMD:D_SMA, B.Cu at (100.6, 139.4)
- added FL2: Choke_CommonMode_PulseElectronics_PH9455x156NL, Inductor_THT:L_CommonMode_PulseElectronics_PH9455xxx6NL_2, F.Cu at (49.2, 110.2)
- added J6: Motor, Connector_Phoenix_MC:PhoenixContact_MCV_1,5_2-G-3.81_1x02_P3.81mm_Vertical, F.Cu at (111.4, 137.5)
- added J7: Conn_02x10_Odd_Even, Connector_IDC:IDC-Header_2x10_P2.54mm_Vertical, F.Cu at (114.6, 98.1)
- added J8: Conn_02x10_Odd_Even, Connector_IDC:IDC-Header_2x10_P2.54mm_Vertical, F.Cu at (134.3, 126.0)
- added J9: Conn_02x10_Odd_Even, Connector_IDC:IDC-Header_2x10_P2.54mm_Vertical, F.Cu at (145.7, 126.0)
- added L1: 33µH, Inductor_SMD:L_Chilisin_BMRB00060650, B.Cu at (92.4, 133.7)
- added Q1: 2N7002E, Package_TO_SOT_SMD:SOT-23, B.Cu at (122.9, 128.7)
- added Q2: 2N7002H, Package_TO_SOT_SMD:SOT-23, B.Cu at (126.7, 128.7)
- added R2: 10K, Resistor_SMD:R_0603_1608Metric, B.Cu at (126.7, 126.0)
- added R3: 100R, Resistor_THT:R_Axial_DIN0204_L3.6mm_D1.6mm_P7.62mm_Horizontal, F.Cu at (133.0, 105.7)
- added R4: 4K7, Resistor_THT:R_Axial_DIN0204_L3.6mm_D1.6mm_P7.62mm_Horizontal, F.Cu at (133.0, 108.3)
- added R5: 4K7, Resistor_THT:R_Axial_DIN0204_L3.6mm_D1.6mm_P7.62mm_Horizontal, F.Cu at (133.0, 110.8)
- added R6: 10K, Resistor_SMD:R_0603_1608Metric, B.Cu at (123.1, 131.4)
- added R7: 10K, Resistor_SMD:R_0603_1608Metric, B.Cu at (126.4, 131.4)
- added RV1: 10D561K, Varistor:RV_Disc_D9mm_W6.1mm_P5mm, F.Cu at (42.9, 125.9)
- added U3: WEMOS_D1_mini, RF_Module:WEMOS_D1_mini_light, F.Cu at (149.5, 94.3)
- DRA1, DRA2: footprint Library:DINRailAdapter_3xM3_PhoenixContact_1201578 -> MountingEquipment:DINRailAdapter_3xM3_PhoenixContact_1201578
- J1: value VDD -> Mains; footprint Connector_Phoenix_MC:PhoenixContact_MC_1,5_2-G-3.81_1x02_P3.81mm_Horizontal -> Connector_Phoenix_MC:PhoenixContact_MCV_1,5_2-G-3.81_1x02_P3.81mm_Vertical
- J2: value Conn_02x10_Odd_Even -> Mains Motor; footprint Connector_IDC:IDC-Header_2x10_P2.54mm_Vertical -> Connector_Phoenix_MC:PhoenixContact_MCV_1,5_2-G-3.81_1x02_P3.81mm_Vertical
- J3: value Mains -> VDD; footprint Connector_Phoenix_MC:PhoenixContact_MC_1,5_2-G-3.81_1x02_P3.81mm_Horizontal -> Connector_Phoenix_MC:PhoenixContact_MCV_1,5_2-G-3.81_1x02_P3.81mm_Vertical
- J4: value Mains Motor -> VDD; footprint Connector_Phoenix_MC:PhoenixContact_MC_1,5_2-G-3.81_1x02_P3.81mm_Horizontal -> Connector_Phoenix_MC:PhoenixContact_MCV_1,5_2-G-3.81_1x02_P3.81mm_Vertical
- J5: footprint Connector_Phoenix_MC:PhoenixContact_MC_1,5_2-G-3.81_1x02_P3.81mm_Horizontal -> Connector_Phoenix_MC:PhoenixContact_MCV_1,5_2-G-3.81_1x02_P3.81mm_Vertical
- JP1, JP2: footprint Library:SolderJumper-3_P1.3mm_Open_Pad1.0x1.5mm no silk -> Connector_PinHeader_2.54mm:PinHeader_1x03_P2.54mm_Vertical
- PS2: value TPP-15-109-D -> HLK-30M09; footprint Converter_ACDC:Converter_ACDC_TRACO_TPP-15-1xx-D_THT -> Converter_ACDC:Converter_ACDC_Hi-Link_HLK-30Mxx
- R1: value 100R -> 10K; footprint Resistor_THT:R_Axial_DIN0204_L3.6mm_D1.6mm_P7.62mm_Horizontal -> Resistor_SMD:R_0603_1608Metric; moved to B.Cu
- U2: value TSR_1-2450 -> LM2675N-5; footprint Converter_DCDC:Converter_DCDC_TRACO_TSR-1_THT -> Package_SO:SOIC-8_3.9x4.9mm_P1.27mm; moved to B.Cu
- moved J1 112.2 mm to (43.5, 150.2), turned to 0 degrees
- moved DRA2 96.7 mm to (35.9, 123.5), turned to 90 degrees
- moved F1 93.4 mm to (45.4, 140.6), turned to 90 degrees
- moved J2 89.4 mm to (54.9, 150.2), turned to 0 degrees
- moved F2 83.2 mm to (56.8, 140.6), turned to 90 degrees
- moved U2 62.0 mm to (101.3, 133.7), turned to -90 degrees
- moved DRA1 55.1 mm to (155.9, 123.5), turned to 90 degrees
- moved PS2 50.9 mm to (86.0, 98.1), turned to -90 degrees
- moved JP2 42.8 mm to (122.9, 123.5)
- moved S1 40.4 mm to (68.1, 134.3), turned to -90 degrees
- moved JP1 39.3 mm to (122.9, 121.0)
- moved J4 38.8 mm to (111.4, 150.2), turned to 0 degrees
- moved J5 33.0 mm to (122.9, 137.5), turned to 0 degrees
- moved R1 30.3 mm to (122.9, 126.0)
- moved J3 22.4 mm to (122.9, 150.2), turned to 0 degrees
Connections:
- F1 pad 2: Net-(PS2-AC/L) -> Net-(C4-Pad1)
- J1 pad 1: VSS -> LINE
- J1 pad 2: VDD -> NEUT
- J2 pad 1: Motor N -> 230V Motor
- J2 pad 2: Motor N -> NEUT
- J3 pad 1: LINE -> VSS
- J3 pad 2: NEUT -> VDD
- J4 pad 1: 230V Motor -> VSS
- J4 pad 2: NEUT -> VDD
- JP1 pad 1: RX0 -> RX/RX0
- JP1 pad 2: RX -> Net-(JP1-C)
- JP1 pad 3: RX1 -> D4/RX1
- JP2 pad 1: TX0 -> TX/TX0
- JP2 pad 2: TX -> Net-(JP2-C)
- JP2 pad 3: TX1 -> D3/TX1
- PS2 pad 1: NEUT -> Net-(PS2-AC/L)
- PS2 pad 2: Net-(PS2-AC/L) -> Net-(PS2-AC/N)
- PS2 pad 3: unconnected-(PS2-Trim-Pad3) -> VSS
- R1 pad 1: En Motor -> Net-(JP1-C)
- R1 pad 2: Net-(S1-+LED) -> +3.3V
- U2 pad 1: VDD -> Net-(U2-CB)
- U2 pad 2: VSS -> unconnected-(U2-NC-Pad2)
- U2 pad 3: VCC -> unconnected-(U2-NC-Pad3)
Routing:
- net +3.3V: track 0.00 -> 89.4 mm, vias 0 -> 2
- net TX/TX0: track 0.00 -> 42.7 mm
- net RX/RX0: track 0.00 -> 35.7 mm
- net D3/TX1: track 0.00 -> 34.2 mm
- net A0: track 0.00 -> 34.0 mm, vias 0 -> 1
- net D1/SCL: track 0.00 -> 33.5 mm
- net Net-(PS2-AC/L): track 8.50 -> 39.7 mm
- net Motor L: track 31.1 -> 0.00 mm
- net D2/SDA: track 0.00 -> 29.9 mm
- net VCC: track 37.7 -> 67.6 mm, vias 0 -> 2
- net Motor N: track 29.8 -> 0.00 mm
- net D5: track 0.00 -> 29.5 mm
- net Net-(C4-Pad1): track 0.00 -> 29.1 mm
- net NEUT: track 35.6 -> 64.0 mm
- net Net-(S1-+LED): track 44.0 -> 72.1 mm
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- added copper zone on B.Cu, net Net-(D1-K)
- added copper zone on B.Cu, net Net-(U2-CB)
- added copper zone on B.Cu, net VCC
- added copper zone on B.Cu, net VDD
Other:
- board size 62.2 x 83.8 mm -> 130.2 x 61 mm
- board text added: "3V3"
- board text added: "5V"
- board text added: "9V"
- board text added: "A0"
- board text added: "AC"
- board text added: "D1"
- board text added: "D2"
- board text added: "D3"
- board text added: "D4"
- board text added: "D5"
- board text added: "D6"
- board text added: "D7"
- board text added: "D8"
- board text added: "GND"
- board text added: "UART"
- board text removed: "0V DC"
- board text removed: "1A"
- board text removed: "42V AC"
- board text removed: "6A"
- board text removed: "9V DC"
- board text removed: "Mains"
- board text removed: "Motor"
- board text removed: "RX"
- board text removed: "SFD Bus"
- board text removed: "TX"
- board text removed: "chrissileinus"
- board text removed: "espSFD"
