File: hardware/pcb/espSFDmains/espSFDmains.kicad_pcb (KiCad board)
At the start: 2 copper layers, 130.2 x 61 mm, 36 parts, among them J1 Mains, J2 Mains Motor, J3 VDD, J4 VDD, J5 Motor, J6 Motor, J7 Conn_02x10_Odd_Even, J8 Conn_02x10_Odd_Even, J9 Conn_02x10_Odd_Even, Q1 2N7002E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

Commit message: ghfd
Routing:
- net NEUT: track 64.0 -> 62.7 mm
Other:
- outline, holes or cut-outs redrawn
Changed lines of the file:
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@@
 	)
 	(gr_line
-		(start 62.164 141.915)
-		(end 62.164 149.535)
+		(start 103.82 102.545)
+		(end 68.26 138.105)
 		(stroke
 			(width 0.1)
@@
 	)
 	(gr_arc
-		(start 66.228 149.535)
-		(mid 64.196 151.567)
-		(end 62.164 149.535)
+		(start 61.91 140.645)
+		(mid 62.200019 139.186976)
+		(end 63.025923 137.950923)
 		(stroke
 			(width 0.1)
@@
 		(layer "Edge.Cuts")
 	)
-	(gr_arc
-		(start 68.26 138.105)
-		(mid 65.466 138.359)
-		(end 65.212 135.565)
+	(gr_line
+		(start 101.125923 99.850924)
+		(end 63.025924 137.950923)
 		(stroke
 			(width 0.1)
@@
 	)
 	(gr_arc
-		(start 97.851 102.926)
-		(mid 100.645 102.926)
-		(end 100.645 105.72)
+		(start 101.125923 99.850922)
+		(mid 103.82 99.850922)
+		(end 103.82 102.545)
+		(stroke
+			(width 0.1)
+			(type solid)
+		)
+		(layer "Edge.Cuts")
+	)
+	(gr_line
+		(start 61.91 140.645)
+		(end 61.91 149.535)
 		(stroke
 			(width 0.1)
@@
 	)
 	(gr_line
-		(start 66.228 141.915)
-		(end 66.228 149.535)
+		(start 65.72 140.645)
+		(end 65.72 149.535)
+		(stroke
+			(width 0.1)
+			(type default)
+		)
+		(layer "Edge.Cuts")
+	)
+	(gr_line
+		(start 65.72 140.645)
+		(end 68.26 138.105)
+		(stroke
+			(width 0.1)
+			(type default)
+		)
+		(layer "Edge.Cuts")
+	)
+	(gr_arc
+		(start 65.72 149.535)
+		(mid 63.815 151.44)
+		(end 61.91 149.535)
 		(stroke
 			(width 0.1)
@@
 		(layer "Edge.Cuts")
 	)
-	(gr_arc
-		(start 62.164 141.915)
-		(mid 64.196 139.883)
-		(end 66.228 141.915)
-		(stroke
-			(width 0.1)
-			(type default)
-		)
-		(layer "Edge.Cuts")
-	)
-	(gr_line
-		(start 68.26 138.105)
-		(end 100.645 105.72)
-		(stroke
-			(width 0.1)
-			(type default)
-		)
-		(layer "Edge.Cuts")
-	)
-	(gr_line
-		(start 65.212001 135.565)
-		(end 97.851 102.926)
-		(stroke
-			(width 0.1)
-			(type default)
-		)
-		(layer "Edge.Cuts")
-	)
 	(gr_text "GND"
 		(at 111.44 145.09 0)
@@
 			)
 			(justify right)
+		)
+	)
+	(dimension
+		(type orthogonal)
+		(layer "User.1")
+		(pts
+			(xy 160.97 93.02) (xy 160.97 153.98)
+		)
+		(height 14.905)
+		(orientation 1)
+		(format
+			(prefix "")
+			(suffix "")
+			(units 3)
+			(units_format 1)
+			(precision 4)
+		)
+		(style
+			(thickness 0.15)
+			(arrow_length 1.27)
+			(text_position_mode 0)
+			(arrow_direction outward)
+			(extension_height 0.58642)
+			(extension_offset 0.5)
+			(keep_text_aligned yes)
+		)
+		(gr_text "60,9600 mm"
+			(at 174.725 123.5 90)
+			(layer "User.1")
+			(effects
+				(font
+					(size 1 1)
+					(thickness 0.15)
+				)
+			)
+		)
+	)
+	(dimension
+		(type orthogonal)
+		(layer "User.1")
+		(pts
+			(xy 30.795 93.02) (xy 160.97 93.02)
+		)
+		(height -19.52)
+		(orientation 0)
+		(format
+			(prefix "")
+			(suffix "")
+			(units 3)
+			(units_format 1)
+			(precision 4)
+		)
+		(style
+			(thickness 0.15)
+			(arrow_length 1.27)
+			(text_position_mode 0)
+			(arrow_direction outward)
+			(extension_height 0.58642)
+			(extension_offset 0.5)
+			(keep_text_aligned yes)
+		)
+		(gr_text "130,1750 mm"
+			(at 95.8825 72.35 0)
+			(layer "User.1")
+			(effects
+				(font
+					(size 1 1)
+					(thickness 0.15)
+				)
+			)
 		)
 	)
@@
 	)
 	(segment
+		(start 47.305 146.955)
+		(end 47.9 146.36)
+		(width 1)
+		(layer "B.Cu")
+		(net 7)
+	)
+	(segment
+		(start 47.9 127.425)
+		(end 51.515 127.425)
+		(width 1)
+		(layer "B.Cu")
+		(net 7)
+	)
+	(segment
+		(start 59.21 114.57)
+		(end 59.21 110.165)
+		(width 1)
+		(layer "B.Cu")
+		(net 7)
+	)
+	(segment
+		(start 61.79 117.15)
+		(end 59.21 114.57)
+		(width 1)
+		(layer "B.Cu")
+		(net 7)
+	)
+	(segment
+		(start 47.305 150.17)
+		(end 47.305 146.955)
+		(width 1)
+		(layer "B.Cu")
+		(net 7)
+	)
+	(segment
 		(start 47.9 127.425)
 		(end 47.9 146.36)
@@
 	)
 	(segment
-		(start 47.9 146.36)
-		(end 47.305 146.36)
+		(start 56.83 146.36)
+		(end 47.9 146.36)
 		(width 1)
 		(layer "B.Cu")
@@
 	)
 	(segment
-		(start 47.305 146.36)
-		(end 47.305 150.17)
+		(start 58.735 148.265)
+		(end 56.83 146.36)
 		(width 1)
 		(layer "B.Cu")
@@
 	)
 	(segment
-		(start 58.735 147.63)
-		(end 57.465 146.36)
-		(width 1)
-		(layer "B.Cu")
-		(net 7)
-	)
-	(segment
-		(start 57.465 146.36)
-		(end 47.305 146.36)
-		(width 1)
-		(layer "B.Cu")
-		(net 7)
-	)
-	(segment
-		(start 47.9 127.425)
-		(end 51.515 127.425)
-		(width 1)
-		(layer "B.Cu")
-		(net 7)
-	)
-	(segment
-		(start 59.21 114.57)
-		(end 59.21 110.165)
-		(width 1)
-		(layer "B.Cu")
-		(net 7)
-	)
-	(segment
-		(start 61.79 117.15)
-		(end 59.21 114.57)
-		(width 1)
-		(layer "B.Cu")
-		(net 7)
-	)
-	(segment
 		(start 58.735 150.17)
-		(end 58.735 147.63)
+		(end 58.735 148.265)
 		(width 1)
 		(layer "B.Cu")
@@
 	)
 	(segment
+		(start 123.49 116.5)
+		(end 117.775 116.5)
+		(width 0.25)
+		(layer "B.Cu")
+		(net 15)
+	)
+	(segment
 		(start 127.95 120.96)
-		(end 122.87 115.88)
+		(end 123.49 116.5)
 		(width 0.25)
 		(layer "B.Cu")
@@
 	)
 	(segment
-		(start 122.87 115.88)
+		(start 117.775 116.5)
 		(end 117.155 115.88)
 		(width 0.25)
@@
 		(polygon
 			(pts
-				(xy 150.81 93.02) (xy 107.63 93.02) (xy 107.63 102.545) (xy 68.26 141.915) (xy 68.26 153.98) (xy 150.81 153.98)
-			)
-		)
+				(xy 150.81 93.02) (xy 105.725 93.02) (xy 105.725 102.545) (xy 66.99 141.28) (xy 66.99 153.98) (xy 150.81 153.98)
+			)
+		)

Commit message: jfgj
Parts:
- removed C4: 0.1uF/275Vac, Capacitor_THT:C_Rect_L16.5mm_W5.0mm_P15.00mm_MKT
- removed FL2: Choke_CommonMode_PulseElectronics_PH9455x156NL, Inductor_THT:L_CommonMode_PulseElectronics_PH9455xxx6NL_2
- removed J6: Motor, Connector_Phoenix_MC:PhoenixContact_MCV_1,5_2-G-3.81_1x02_P3.81mm_Vertical
- removed J7: Conn_02x10_Odd_Even, Connector_IDC:IDC-Header_2x10_P2.54mm_Vertical
- removed RV1: 10D561K, Varistor:RV_Disc_D9mm_W6.1mm_P5mm
- added J10: Conn_01x04_Socket, Connector_Phoenix_MC:PhoenixContact_MCV_1,5_4-G-3.81_1x04_P3.81mm_Vertical, F.Cu at (93.0, 152.1)
- added J11: Conn_01x04_Socket, Connector_Phoenix_MC:PhoenixContact_MCV_1,5_4-G-3.81_1x04_P3.81mm_Vertical, F.Cu at (93.0, 139.4)
- added JP3: SolderJumper_2_Open, Jumper:SolderJumper-2_P1.3mm_Open_Pad1.0x1.5mm, F.Cu at (143.8, 98.1)
- added JP4: SolderJumper_2_Open, Jumper:SolderJumper-2_P1.3mm_Open_Pad1.0x1.5mm, F.Cu at (143.8, 100.6)
- J4: value VDD -> Conn_01x04_Socket; footprint Connector_Phoenix_MC:PhoenixContact_MCV_1,5_2-G-3.81_1x02_P3.81mm_Vertical -> Connector_Phoenix_MC:PhoenixContact_MCV_1,5_4-G-3.81_1x04_P3.81mm_Vertical
- J5: footprint Connector_Phoenix_MC:PhoenixContact_MCV_1,5_2-G-3.81_1x02_P3.81mm_Vertical -> Connector_Phoenix_MC:PhoenixContact_MCV_1,5_4-G-3.81_1x04_P3.81mm_Vertical
- JP1, JP2: footprint Connector_PinHeader_2.54mm:PinHeader_1x03_P2.54mm_Vertical -> Jumper:SolderJumper-3_P1.3mm_Open_Pad1.0x1.5mm
- R3, R4, R5: footprint Resistor_THT:R_Axial_DIN0204_L3.6mm_D1.6mm_P7.62mm_Horizontal -> Resistor_SMD:R_0603_1608Metric; moved to B.Cu
- moved R3 59.8 mm to (77.8, 128.6)
- moved J5 49.8 mm to (75.2, 152.1)
- moved C1 45.2 mm to (98.1, 98.7), turned to 90 degrees
- moved D1 41.9 mm to (93.7, 98.1), turned to 90 degrees
- moved U2 38.6 mm to (87.9, 97.5), turned to 0 degrees
- moved J4 37.8 mm to (75.2, 139.4)
- moved PS2 37.7 mm to (51.5, 113.3), turned to 0 degrees
- moved U3 36.2 mm to (113.3, 93.0), turned to 0 degrees
- moved JP1 34.9 mm to (143.8, 148.9), turned to 180 degrees
- moved C3 34.0 mm to (81.6, 98.7), turned to 90 degrees
- moved C2 33.8 mm to (87.9, 101.3), turned to 0 degrees
- moved R1 33.7 mm to (145.7, 150.8), turned to 90 degrees
- moved JP2 31.0 mm to (143.8, 146.4), turned to 180 degrees
- moved Q1 29.6 mm to (142.6, 150.8), turned to 180 degrees
- moved R2 28.3 mm to (145.7, 147.0), turned to 90 degrees
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Connections:
- F1 pad 2: Net-(C4-Pad1) -> Net-(PS2-AC/L)
- J1 pad 1: LINE -> NEUT
- J1 pad 2: NEUT -> LINE
- J2 pad 1: 230V Motor -> NEUT
- J2 pad 2: NEUT -> 230V Motor
- J4 pad 2: VDD -> VCC
- J5 pad 2: Motor L -> Motor N
- PS2 pad 2: Net-(PS2-AC/N) -> NEUT
- R4 pad 2: D1/SCL -> Net-(JP3-A)
- R5 pad 2: D2/SDA -> Net-(JP4-A)
- U3 pad 2: A0 -> unconnected-(U3-A0-Pad2)
- U3 pad 6: D7 -> unconnected-(U3-MOSI/D7-Pad6)
- U3 pad 7: D8 -> unconnected-(U3-CS/D8-Pad7)
Routing:
- net Motor N: track 0.00 -> 111.4 mm
- net Motor L: track 0.00 -> 102.0 mm
- net +3.3V: track 89.4 -> 11.7 mm, vias 2 -> 3
- net VDD: track 84.3 -> 14.2 mm, vias 0 -> 6
- net Net-(S1-+LED): track 72.1 -> 2.62 mm
- net D4/RX1: track 23.6 -> 93.0 mm, vias 0 -> 1
- net VCC: track 67.6 -> 2.16 mm, vias 2 -> 17
- net D3/TX1: track 34.2 -> 96.8 mm, vias 0 -> 1
- net D1/SCL: track 33.5 -> 77.3 mm, vias 0 -> 1
- net D2/SDA: track 29.9 -> 73.1 mm, vias 0 -> 1
- net A0: track 34.0 -> 0.00 mm, vias 1 -> 0
- net En Motor: track 16.2 -> 47.4 mm
- net RX/RX0: track 35.7 -> 64.9 mm, vias 0 -> 1
- net Net-(C4-Pad1): track 29.1 -> 0.00 mm
- net TX/TX0: track 42.7 -> 65.9 mm, vias 0 -> 1
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- added copper zone on In1.Cu, net +3.3V
- added copper zone on B.Cu, net Motor L
- added copper zone on B.Cu, net Motor N
- added copper zone on In2.Cu, net VCC
- added copper zone on In1.Cu, net VDD
- removed copper zone on F.Cu, net Motor L
- removed copper zone on F.Cu, net Motor N
- removed copper zone on B.Cu, net VDD
Other:
- board size 130.2 x 61 mm -> 111.8 x 63.5 mm
- copper layers 2 -> 4
- board text added: "I²C Pull Up"
- board text added: "Mains 230V"
- board text added: "Motor 42V/AC"
- board text added: "Motor AC"
- board text added: "RX"
- board text added: "SCL"
- board text added: "SDA"
- board text added: "SFD Bus Power"
- board text added: "TX"
- board text removed: "3V3"
- board text removed: "A0"
- board text removed: "AC"
- board text removed: "D7"
- board text removed: "D8"

Commit message: frhgfd
Parts:
- removed Q1: 2N7002E, Package_TO_SOT_SMD:SOT-23
- removed Q2: 2N7002H, Package_TO_SOT_SMD:SOT-23
- removed R1, R2, R6, R7: 10K, Resistor_SMD:R_0603_1608Metric
- added C4: 100nF/50V, Capacitor_SMD:C_0603_1608Metric, B.Cu at (115.9, 99.4)
- added C5: 100nF/50V, Capacitor_SMD:C_0603_1608Metric, B.Cu at (123.5, 99.4)
- added REF**: Symbol_HighVoltage_Triangle_6x6mm_Copper, Symbol:Symbol_HighVoltage_Triangle_6x6mm_Copper, F.Cu at (42.2, 150.2)
- added REF**: OSHW-Symbol_6.7x6mm_SilkScreen, Symbol:OSHW-Symbol_6.7x6mm_SilkScreen, F.Cu at (112.7, 138.7)
- added REF**: Symbol_HighVoltage_Triangle_6x6mm_Copper, Symbol:Symbol_HighVoltage_Triangle_6x6mm_Copper, B.Cu at (42.2, 150.2)
- added U1: TXS0102DCT, Package_SO:SSOP-8_2.95x2.8mm_P0.65mm, B.Cu at (119.7, 99.4)
- J10: value Conn_01x04_Socket -> D1 & D2
- J11: value Conn_01x04_Socket -> D3 & D4
- J4: value Conn_01x04_Socket -> D5 & D6
- J8, J9: value Conn_02x10_Odd_Even -> SFD Bus
- moved JP2 54.0 mm to (119.7, 98.1)
- moved JP1 54.0 mm to (119.7, 100.6)
- moved JP3 14.0 mm to (129.9, 98.1), turned to 0 degrees
- moved JP4 14.0 mm to (129.9, 100.6), turned to 0 degrees
- moved R4 14.0 mm to (129.9, 98.1), turned to 180 degrees
- moved R5 14.0 mm to (129.9, 100.6), turned to 180 degrees
- moved J8 1.27 mm to (122.2, 127.3)
- moved J9 1.27 mm to (133.7, 127.3)
Connections:
- U3 pad 6: unconnected-(U3-MOSI/D7-Pad6) -> Enable UART
Routing:
- net RX: track 21.7 -> 96.4 mm
- net TX: track 21.7 -> 83.6 mm
- net TX/TX0: track 65.9 -> 17.3 mm, vias 1 -> 0
- net RX/RX0: track 64.9 -> 17.3 mm, vias 1 -> 0
- net D4/RX1: track 93.0 -> 67.4 mm, vias 1 -> 0
- net D3/TX1: track 96.8 -> 75.7 mm, vias 1 -> 2
- net Enable UART: track 0.00 -> 8.57 mm
- net +3.3V: track 11.7 -> 6.67 mm, vias 3 -> 2
- net VSS: track 0.00 -> 2.49 mm, vias 22 -> 24
- net Motor N: track 111.4 -> 109.0 mm
- net Net-(JP2-C): track 5.74 -> 3.55 mm
- net Motor L: track 102.0 -> 100.2 mm
- net VCC: track 2.16 -> 3.62 mm
- net Net-(JP1-C): track 5.28 -> 3.99 mm
- net D2/SDA: track 73.1 -> 71.9 mm
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Other:
- board text added: "SFD Data-Bus & Power"
- board text added: "UART Select"
- board text added: "espSFDmains"
- board text removed: "SFD Bus Power"
- board text removed: "UART"

Commit message: fhdgfh
Parts:
- removed REF** (x2): Symbol_HighVoltage_Triangle_6x6mm_Copper, Symbol:Symbol_HighVoltage_Triangle_6x6mm_Copper
- removed REF**: OSHW-Symbol_6.7x6mm_SilkScreen, Symbol:OSHW-Symbol_6.7x6mm_SilkScreen
- added D2: LESD5D5.0CT1G, Diode_SMD:D_SOD-523, B.Cu at (105.7, 130.5)
- added D3: LESD5D5.0CT1G, Diode_SMD:D_SOD-523, B.Cu at (108.3, 130.5)
- added D4: LESD5D5.0CT1G, Diode_SMD:D_SOD-523, B.Cu at (110.8, 130.5)
- added D5: LESD5D5.0CT1G, Diode_SMD:D_SOD-523, B.Cu at (103.2, 130.5)
- added D6: LESD5D5.0CT1G, Diode_SMD:D_SOD-523, B.Cu at (82.9, 130.5)
- added D7: LESD5D5.0CT1G, Diode_SMD:D_SOD-523, B.Cu at (86.7, 130.5)
- added D8: LESD5D5.0CT1G, Diode_SMD:D_SOD-523, B.Cu at (129.2, 150.8)
- added D9: LESD5D5.0CT1G, Diode_SMD:D_SOD-523, B.Cu at (129.2, 147.0)
- JP1: value SolderJumper_3_Open -> RX Select
- JP2: value SolderJumper_3_Open -> TX Select
Connections:
- net Net-(D1-K) renamed /VSW
- net Net-(JP1-C) renamed RX Selected
- net Net-(JP2-C) renamed TX Selected
- net Net-(U2-CB) renamed /CB
- net VCC renamed +5V
- net VDD renamed +9V
- net VSS renamed GND
Routing:
- net +9V: track 14.2 -> 0.00 mm, vias 6 -> 7
- net +5V: vias 17 -> 6
- added copper zone on B.Cu, net +9V

Commit message: hedfhf
Routing:
- net Motor N: track 109.0 -> 0.00 mm
- net Motor L: track 100.2 -> 0.00 mm
Changed lines of the file:
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@@
-	)
-	(segment
-		(start 117.155 140.01)
-		(end 122.235 134.93)
-		(width 2.25)
-		(layer "B.Cu")
-		(net 1)
-	)
-	(segment
-		(start 89.85 146.995)
-		(end 88.58 146.995)
-		(width 2.25)
-		(layer "B.Cu")
-		(net 1)
-	)
-	(segment
-		(start 86.675 148.9)
-		(end 86.675 152.075)
-		(width 2.25)
-		(layer "B.Cu")
-		(net 1)
-	)
-	(segment
-		(start 86.675 148.9)
-		(end 86.675 146.995)
-		(width 2.25)
-		(layer "B.Cu")
-		(net 1)
-	)
-	(segment
-		(start 89.85 146.995)
-		(end 86.675 146.995)
-		(width 2.25)
-		(layer "B.Cu")
-		(net 1)
-	)
-	(segment
-		(start 122.235 134.93)
-		(end 122.235 140.01)
-		(width 2.25)
-		(layer "B.Cu")
-		(net 1)
-	)
-	(segment
-		(start 110.17 146.995)
-		(end 117.155 140.01)
-		(width 2.25)
-		(layer "B.Cu")
-		(net 1)
-	)
-	(segment
-		(start 136.205 140.01)
-		(end 122.235 140.01)
-		(width 2.25)
-		(layer "B.Cu")
-		(net 1)
-	)
-	(segment
-		(start 122.235 140.01)
-		(end 117.155 140.01)
-		(width 2.25)
-		(layer "B.Cu")
-		(net 1)
-	)
-	(segment
-		(start 122.235 134.93)
-		(end 136.205 134.93)
-		(width 2.25)
-		(layer "B.Cu")
-		(net 1)
-	)
-	(segment
-		(start 82.865 149.535)
-		(end 82.865 152.075)
-		(width 2.25)
-		(layer "B.Cu")
-		(net 1)
-	)
-	(segment
-		(start 89.85 146.995)
-		(end 110.17 146.995)
-		(width 2.25)
-		(layer "B.Cu")
-		(net 1)
-	)
-	(segment
-		(start 88.58 146.995)
-		(end 86.675 148.9)
-		(width 2.25)
-		(layer "B.Cu")
-		(net 1)
-	)
-	(segment
-		(start 86.675 146.995)
-		(end 85.405 146.995)
-		(width 2.25)
-		(layer "B.Cu")
-		(net 1)
-	)
-	(segment
-		(start 136.205 134.93)
-		(end 136.205 140.01)
-		(width 2.25)
-		(layer "B.Cu")
-		(net 1)
-	)
-	(segment
-		(start 85.405 146.995)
-		(end 82.865 149.535)
-		(width 2.25)
-		(layer "B.Cu")
-		(net 1)
-	)
-	(segment
-		(start 79.055 149.535)
-		(end 84.262 144.328)
-		(width 2.25)
-		(layer "B.Cu")
-		(net 2)
-	)
-	(segment
-		(start 122.235 131.12)
-		(end 122.235 127.31)
-		(width 2.25)
-		(layer "B.Cu")
-		(net 2)
-	)
-	(segment
-		(start 75.245 150.4875)
-		(end 75.245 152.075)
-		(width 2.25)
-		(layer "B.Cu")
-		(net 2)
-	)
-	(segment
-		(start 79.055 152.075)
-		(end 79.055 149.535)
-		(width 2.25)
-		(layer "B.Cu")
-		(net 2)
-	)
-	(segment
-		(start 120.965 132.39)
-		(end 122.235 131.12)
-		(width 2.25)
-		(layer "B.Cu")
-		(net 2)
-	)
-	(segment
-		(start 122.235 127.31)
-		(end 136.205 127.31)
-		(width 2.25)
-		(layer "B.Cu")
-		(net 2)
-	)
-	(segment
-		(start 109.027 144.328)
-		(end 120.965 132.39)
-		(width 2.25)
-		(layer "B.Cu")
-		(net 2)
-	)
-	(segment
-		(start 136.205 132.39)
-		(end 122.235 132.39)
-		(width 2.25)
-		(layer "B.Cu")
-		(net 2)
-	)
-	(segment
-		(start 81.4045 144.328)
-		(end 75.245 150.4875)
-		(width 2.25)
-		(layer "B.Cu")
-		(net 2)
-	)
-	(segment
-		(start 136.205 127.31)
-		(end 136.205 132.39)
-		(width 2.25)
-		(layer "B.Cu")
-		(net 2)
-	)
-	(segment
-		(start 122.235 132.39)
-		(end 122.235 131.12)
-		(width 2.25)
-		(layer "B.Cu")
-		(net 2)
-	)
-	(segment
-		(start 84.262 144.328)
-		(end 109.027 144.328)
-		(width 2.25)
-		(layer "B.Cu")
-		(net 2)
-	)
-	(segment
-		(start 120.965 132.39)
-		(end 122.235 132.39)
-		(width 2.25)
-		(layer "B.Cu")
-		(net 2)
-	)
-	(segment
-		(start 87.437 144.328)
-		(end 81.4045 144.328)
-		(width 2.25)
-		(layer "B.Cu")
-		(net 2)
 	)
 	(segment
@@
 	)
 	(zone
-		(net 2)
-		(net_name "Motor N")
-		(layer "B.Cu")
-		(hatch edge 0.5)
-		(priority 4)
-		(connect_pads yes
-			(clearance 0.2)
-		)
-		(min_thickness 0.25)
-		(filled_areas_thickness no)
-		(fill yes
-			(thermal_gap 0.5)
-			(thermal_bridge_width 0.5)
-		)
-		(polygon
-			(pts
-				(xy 122.235 127.31) (xy 122.235 132.39) (xy 136.205 132.39) (xy 136.205 127.31)
-			)
-		)
-	)
-	(zone
 		(net 10)
 		(net_name "+9V")
@@
 		(layer "B.Cu")
 		(hatch edge 0.5)
-		(priority 4)
-		(connect_pads yes
-			(clearance 0.2)
-		)
-		(min_thickness 0.25)
-		(filled_areas_thickness no)
-		(fill yes
-			(thermal_gap 0.5)
-			(thermal_bridge_width 0.5)
-		)
-		(polygon
-			(pts
-				(xy 122.235 134.93) (xy 136.205 134.93) (xy 136.205 140.01) (xy 117.155 140.01)
-			)
-		)
-	)
-	(zone
-		(net 31)
-		(net_name "+5V")
-		(layer "B.Cu")
-		(hatch edge 0.5)
-		(priority 1)
+		(priority 7)
 		(connect_pads yes
 			(clearance 0.2)
@@
 		(polygon
 			(pts
+				(xy 137.221 133.787) (xy 121.6 133.787) (xy 110.17 145.217) (xy 85.405 145.217) (xy 81.468 149.154)
+				(xy 81.468 154.107) (xy 88.072 154.107) (xy 88.072 149.154) (xy 89.723 147.503) (xy 111.313 147.503)
+				(xy 117.79 141.026) (xy 137.221 141.026)
+			)
+		)
+	)
+	(zone
+		(net 31)
+		(net_name "+5V")
+		(layer "B.Cu")
+		(hatch edge 0.5)
+		(priority 1)
+		(connect_pads yes
+			(clearance 0.2)
+		)
+		(min_thickness 0.25)
+		(filled_areas_thickness no)
+		(fill yes
+			(thermal_gap 0.5)
+			(thermal_bridge_width 0.5)
+			(smoothing fillet)
+			(radius 0.25)
+		)
+		(polygon
+			(pts
 				(xy 87.818 109.911) (xy 84.135 109.911) (xy 80.071 105.847) (xy 80.071 99.751) (xy 83.119 96.83)
 				(xy 83.119 95.687) (xy 83.119 95.052) (xy 86.675 95.052) (xy 86.675 96.068) (xy 84.4525 96.068)
@@
 			)
 		)
+	)
+	(zone
+		(net 2)
+		(net_name "Motor N")
+		(layer "B.Cu")
+		(hatch edge 0.5)
+		(priority 3)
+		(connect_pads yes
+			(clearance 0.2)
+		)
+		(min_thickness 0.25)
+		(filled_areas_thickness no)
+		(fill yes
+			(thermal_gap 0.5)
+			(thermal_bridge_width 0.5)
+			(smoothing fillet)
+			(radius 0.25)
+		)
+		(polygon
+			(pts
+				(xy 137.221 133.533) (xy 137.221 126.294) (xy 121.092 126.294) (xy 121.092 130.485) (xy 108.9 142.677)
+				(xy 81.214 142.677) (xy 73.721 150.17) (xy 73.721 154.107) (xy 80.325 154.107) (xy 80.325 149.916)
+				(xy 85.278 144.963) (xy 110.043 144.963) (xy 121.473 133.533)
+			)
+		)
