File: hardware/pcb/espSFDmains/espSFDmains.kicad_pcb (KiCad board)
At the start: 4 copper layers, 111.8 x 63.5 mm, 40 parts, among them J1 Mains, J10 D1 & D2, J11 D3 & D4, J2 Mains Motor, J3 VDD, J4 D5 & D6, J5 Motor, J8 SFD Bus, J9 SFD Bus, U1 TXS0102DCT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

Commit message: vncvn
Parts:
- added JP5: RX Select, Jumper:SolderJumper-3_P1.3mm_Open_Pad1.0x1.5mm, F.Cu at (119.7, 105.7)
- added kibuzzard-6985EF3E: G***, kibuzzard-6985EF3E, F.Cu at (89.8, 152.7)
- added kibuzzard-6985EF3E: G***, kibuzzard-6985EF3E, F.Cu at (104.4, 152.7)
- added kibuzzard-6985EF3E: G***, kibuzzard-6985EF3E, F.Cu at (89.8, 134.9)
- added kibuzzard-6985EF3E: G***, kibuzzard-6985EF3E, F.Cu at (75.2, 152.7)
- added kibuzzard-6985EF47: G***, kibuzzard-6985EF47, F.Cu at (104.4, 148.9)
- added kibuzzard-6985EF47: G***, kibuzzard-6985EF47, F.Cu at (75.2, 148.9)
- added kibuzzard-6985EF47: G***, kibuzzard-6985EF47, F.Cu at (89.7, 148.9)
- added kibuzzard-6985EF5B: G***, kibuzzard-6985EF5B, F.Cu at (42.9, 148.9)
- added kibuzzard-6985EF62: G***, kibuzzard-6985EF62, F.Cu at (42.9, 152.7)
- added kibuzzard-6985EF84: G***, kibuzzard-6985EF84, F.Cu at (57.5, 148.9)
- added kibuzzard-6985EF8A: G***, kibuzzard-6985EF8A, F.Cu at (57.5, 152.7)
- added kibuzzard-6985F184: G***, kibuzzard-6985F184, F.Cu at (90.1, 141.3)
- added kibuzzard-6985F19C: G***, kibuzzard-6985F19C, F.Cu at (90.1, 145.1)
- added kibuzzard-6985F1A9: G***, kibuzzard-6985F1A9, F.Cu at (75.5, 141.3)
- added kibuzzard-6985F1B7: G***, kibuzzard-6985F1B7, F.Cu at (75.5, 145.1)
- added kibuzzard-6985F1DD: G***, kibuzzard-6985F1DD, F.Cu at (104.7, 141.3)
- added kibuzzard-6985F1E4: G***, kibuzzard-6985F1E4, F.Cu at (104.8, 145.1)
- added kibuzzard-6985F203: G***, kibuzzard-6985F203, F.Cu at (89.8, 131.1)
- added kibuzzard-6985F28B: G***, kibuzzard-6985F28B, F.Cu at (104.4, 128.6)
- added kibuzzard-6985F291: G***, kibuzzard-6985F291, F.Cu at (104.4, 133.0)
- added kibuzzard-6985F35C: G***, kibuzzard-6985F35C, F.Cu at (75.3, 139.3)
- added kibuzzard-6985F37C: G***, kibuzzard-6985F37C, F.Cu at (104.5, 139.3)
- added kibuzzard-6985F37C: G***, kibuzzard-6985F37C, F.Cu at (89.9, 139.3)
- added kibuzzard-6985F394: G***, kibuzzard-6985F394, F.Cu at (89.9, 136.8)
- added kibuzzard-6985F3A9: G***, kibuzzard-6985F3A9, F.Cu at (104.5, 136.9)
- added kibuzzard-6985F3D8: G***, kibuzzard-6985F3D8, F.Cu at (58.0, 145.5)
- added kibuzzard-6985F3ED: G***, kibuzzard-6985F3ED, F.Cu at (42.9, 145.4)
- added kibuzzard-6985F472: G***, kibuzzard-6985F472, F.Cu at (129.8, 121.3)
- added kibuzzard-6985F4E1: G***, kibuzzard-6985F4E1, F.Cu at (116.5, 99.4)
- added kibuzzard-6985F4F7: G***, kibuzzard-6985F4F7, F.Cu at (122.9, 99.4)
- added kibuzzard-6985F567: G***, kibuzzard-6985F567, F.Cu at (119.7, 95.9)
- added kibuzzard-6985F5B0: G***, kibuzzard-6985F5B0, F.Cu at (119.7, 103.5)
- added kibuzzard-6985F603: G***, kibuzzard-6985F603, F.Cu at (122.2, 107.6)
- added kibuzzard-6985F68A: G***, kibuzzard-6985F68A, F.Cu at (118.1, 107.6)
- added kibuzzard-6985F70D: G***, kibuzzard-6985F70D, F.Cu at (129.9, 95.9)
- moved J5 40.6 mm to (112.1, 134.9), turned to 90 degrees
- moved J4 39.2 mm to (112.1, 152.7), turned to 90 degrees
- moved D2 29.8 mm to (79.4, 144.5)
- moved D6 28.1 mm to (108.6, 141.9), turned to 90 degrees
- moved D5 26.4 mm to (79.4, 141.9), turned to 90 degrees
- moved D7 26.0 mm to (108.6, 144.5)
- moved D4 21.9 mm to (94.0, 144.5)
- moved J3 21.7 mm to (97.5, 134.9), turned to 90 degrees
- moved D3 18.3 mm to (94.0, 141.9), turned to 90 degrees
- moved J11 14.1 mm to (97.5, 152.7), turned to 90 degrees
- moved J10 10.2 mm to (82.9, 152.7), turned to 90 degrees
- moved J2 3.86 mm to (65.1, 152.7), turned to 90 degrees
- moved J8 1.27 mm to (123.5, 127.3)
- moved J1 0.90 mm to (50.5, 152.7), turned to 90 degrees
- moved D8 0.63 mm to (129.9, 150.8)
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Connections:
- J10 pad 3: D1/SCL -> D2/SDA
- J10 pad 4: D2/SDA -> D1/SCL
- J11 pad 3: D3/TX1 -> D4/RX1
- J11 pad 4: D4/RX1 -> D3/TX1
- J4 pad 3: D5 -> D6
- J4 pad 4: D6 -> D5
- J5 pad 1: Motor N -> Motor L
- J5 pad 2: Motor N -> Motor L
- J5 pad 3: Motor L -> Motor N
- J5 pad 4: Motor L -> Motor N
- U1 pad 6: Enable UART -> OE
Routing:
- net D4/RX1: track 67.8 -> 90.4 mm, vias 0 -> 2
- net D3/TX1: track 76.1 -> 93.7 mm, vias 2 -> 0
- net D2/SDA: track 71.9 -> 86.6 mm, vias 1 -> 0
- net D1/SCL: track 76.0 -> 84.9 mm, vias 1 -> 0
- net OE: track 0.00 -> 8.30 mm, vias 0 -> 1
- net LINE: track 26.0 -> 21.3 mm
- net D6: track 47.2 -> 51.6 mm, vias 0 -> 2
- net Enable UART: track 8.57 -> 5.05 mm
- net 230V Motor: track 11.0 -> 7.78 mm
- net D5: track 51.4 -> 48.5 mm, vias 0 -> 2
- net Net-(JP4-A): track 2.34 -> 0.00 mm
- net Net-(JP3-A): track 2.34 -> 0.00 mm
- net RX Selected: track 3.99 -> 1.95 mm
- net NEUT: track 49.7 -> 51.6 mm
- net +3.3V: track 6.67 -> 5.33 mm, vias 2 -> 3
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Other:
- board text removed: "0"
- board text removed: "1"
- board text removed: "5V"
- board text removed: "9V"
- board text removed: "D1"
- board text removed: "D2"
- board text removed: "D3"
- board text removed: "D4"
- board text removed: "D5"
- board text removed: "D6"
- board text removed: "GND"
- board text removed: "I²C Pull Up"
- board text removed: "Mains 230V"
- board text removed: "Motor 42V/AC"
- board text removed: "Motor AC"
- board text removed: "N"
- board text removed: "RX"
- board text removed: "SCL"
- board text removed: "SDA"
- board text removed: "SFD Data-Bus & Power"
- board text removed: "TX"
- board text removed: "UART Select"

Commit message: ffd hdf
Parts:
- added C6: 68µF/16V, Capacitor_Tantalum_SMD:CP_EIA-7343-43_Kemet-X, B.Cu at (133.0, 115.9)
- added C7: 15µF/50V, Capacitor_Tantalum_SMD:CP_EIA-7343-43_Kemet-X, B.Cu at (118.4, 146.4)
- added C8: 68µF/16V, Capacitor_Tantalum_SMD:CP_EIA-7343-43_Kemet-X, B.Cu at (82.2, 115.2)
- added U4: NCP1117-3.3_SOT223, Package_TO_SOT_SMD:SOT-223-3_TabPin2, B.Cu at (79.1, 108.3)
- DRA1: moved to B.Cu
Connections:
- J10 pad 2: +5V -> +3.3V
- J11 pad 2: +5V -> +3.3V
- J4 pad 2: +5V -> +3.3V
- U3 pad 8: +3.3V -> unconnected-(U3-3V3-Pad8)
Routing:
- net +3.3V: track 5.33 -> 14.2 mm, vias 3 -> 6
- net +9V: track 0.00 -> 8.88 mm
- net +5V: track 2.49 -> 7.60 mm
- net GND: vias 23 -> 35

Commit message: dgs
Parts:
- removed C6: 68µF/16V, Capacitor_Tantalum_SMD:CP_EIA-7343-43_Kemet-X
- removed C7: 15µF/50V, Capacitor_Tantalum_SMD:CP_EIA-7343-43_Kemet-X
- removed kibuzzard-6985EF47 (x3): G***, kibuzzard-6985EF47
- added kibuzzard-69955068: G***, kibuzzard-69955068, F.Cu at (75.2, 148.9)
- added kibuzzard-6995506F: G***, kibuzzard-6995506F, F.Cu at (89.7, 148.9)
- added kibuzzard-69955074: G***, kibuzzard-69955074, F.Cu at (104.4, 148.9)
- U2: value LM2675N-5 -> LM2675M-3.3
- U4: value NCP1117-3.3_SOT223 -> NCP1117-5.0_SOT223
- moved U4 55.6 mm to (133.0, 121.6), turned to 0 degrees
- moved C8 50.8 mm to (133.0, 115.2), turned to 180 degrees
Connections:
- C3 pad 1: +5V -> +3.3V
- C8 pad 1: +3.3V -> +5V
- L1 pad 2: +5V -> +3.3V
- U2 pad 4: +5V -> +3.3V
- U4 pad 2: +3.3V -> +5V
- U4 pad 3: +5V -> +9V
Routing:
- net +5V: track 7.60 -> 19.6 mm, vias 6 -> 1
- net +3.3V: track 14.2 -> 5.33 mm, vias 6 -> 8
- net +9V: track 8.88 -> 0.00 mm, vias 7 -> 11
- net GND: vias 35 -> 32
- added copper zone on B.Cu, net +3.3V
- added copper zone on In2.Cu, net +3.3V
- added copper zone on In1.Cu, net +5V
- removed copper zone on In1.Cu, net +3.3V
- removed copper zone on B.Cu, net +5V
- removed copper zone on In2.Cu, net +5V
