File: hardware/pcb/espSFDmains/espSFDmains.kicad_pcb (KiCad board)
At the start: 4 copper layers, 111.8 x 63.5 mm, 78 parts, among them J1 Mains, J10 D1 & D2, J11 D3 & D4, J2 Mains Motor, J3 VDD, J4 D5 & D6, J5 Motor, J8 SFD Bus, J9 SFD Bus, U1 TXS0102DCT, U2 LM2675M-3.3, U3 WEMOS_D1_mini, U4 NCP1117-5.0_SOT223

Commit message: fhgfds hds
Parts:
- removed PS2: HLK-30M09, Converter_ACDC:Converter_ACDC_Hi-Link_HLK-30Mxx
- removed kibuzzard-6985F28B: G***, kibuzzard-6985F28B
- removed kibuzzard-6985F291: G***, kibuzzard-6985F291
- added PS1: TPP_30-109-D, lib:TPP_30-109-D, F.Cu at (70.2, 111.0)
- DRA1: moved to F.Cu
- moved J3 77.8 mm to (168.0, 167.9)
- moved kibuzzard-6985EF3E 77.8 mm to (160.3, 167.9)
- moved kibuzzard-6985F203 77.8 mm to (160.2, 164.1)
- moved kibuzzard-6985F394 74.4 mm to (160.4, 160.6)
- moved kibuzzard-6985F3A9 47.3 mm to (60.7, 154.7)
- moved J5 47.3 mm to (68.3, 152.7)
- moved C1 22.9 mm to (98.7, 121.6)
- moved C2 22.9 mm to (88.6, 124.1)
- moved C3 22.9 mm to (82.2, 121.6)
- moved D1 22.9 mm to (94.3, 121.0)
- moved L1 22.9 mm to (88.6, 129.2)
- moved U2 22.9 mm to (88.6, 120.3)
- moved F1 12.7 mm to (39.0, 142.6)
- moved DRA2 12.7 mm to (29.5, 123.5)
- moved kibuzzard-6985EF84 11.4 mm to (46.0, 148.9)
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Routing:
- net NEUT: track 51.6 -> 0.00 mm
- net Net-(PS1-LINE): track 26.0 -> 0.00 mm
- net LINE: track 21.3 -> 0.00 mm
- net En Motor: track 47.4 -> 63.6 mm
- net Net-(S1-+LED): track 2.62 -> 15.5 mm
- net 230V Motor: track 7.78 -> 0.00 mm
- net Net-(S1-AC_LOAD2): track 6.61 -> 0.00 mm
- net D6: track 51.6 -> 49.6 mm
- net D4/RX1: track 90.4 -> 88.6 mm
- net D5: track 48.5 -> 49.8 mm
- net D2/SDA: track 86.6 -> 85.4 mm
- net D3/TX1: track 93.7 -> 93.0 mm
- added copper zone on F.Cu, net Motor L
- added copper zone on F.Cu, net Motor N
- removed copper zone on B.Cu, net Motor L
- removed copper zone on B.Cu, net Motor N
Other:
- board size 111.8 x 63.5 mm -> 124.5 x 63.5 mm

Commit message: ffg dsfb
Parts:
- removed JP3, JP4: SolderJumper_2_Open, Jumper:SolderJumper-2_P1.3mm_Open_Pad1.0x1.5mm
- removed kibuzzard-6985EF3E (x4): G***, kibuzzard-6985EF3E
- removed kibuzzard-6985F184: G***, kibuzzard-6985F184
- removed kibuzzard-6985F19C: G***, kibuzzard-6985F19C
- removed kibuzzard-6985F1A9: G***, kibuzzard-6985F1A9
- removed kibuzzard-6985F1B7: G***, kibuzzard-6985F1B7
- removed kibuzzard-6985F1DD: G***, kibuzzard-6985F1DD
- removed kibuzzard-6985F1E4: G***, kibuzzard-6985F1E4
- removed kibuzzard-6985F203: G***, kibuzzard-6985F203
- removed kibuzzard-6985F35C: G***, kibuzzard-6985F35C
- removed kibuzzard-6985F37C (x2): G***, kibuzzard-6985F37C
- removed kibuzzard-6985F3A9: G***, kibuzzard-6985F3A9
- removed kibuzzard-6985F3D8: G***, kibuzzard-6985F3D8
- removed kibuzzard-6985F3ED: G***, kibuzzard-6985F3ED
- removed kibuzzard-6985F70D: G***, kibuzzard-6985F70D
- removed kibuzzard-69955068: G***, kibuzzard-69955068
- removed kibuzzard-6995506F: G***, kibuzzard-6995506F
- removed kibuzzard-69955074: G***, kibuzzard-69955074
- added BT1: Battery_Cell, Battery:BatteryHolder_Keystone_3034_1x20mm, B.Cu at (82.2, 101.3)
- added C6: 100nF/50V, Capacitor_SMD:C_0603_1608Metric, B.Cu at (108.9, 104.8)
- added C7: 1µF/50V, Capacitor_SMD:C_0603_1608Metric, B.Cu at (108.9, 101.6)
- added C9: 10µF/25V, Capacitor_SMD:C_0603_1608Metric, B.Cu at (125.4, 115.9)
- added U5: DS3231MZ, Package_SO:SOIC-8_3.9x4.9mm_P1.27mm, B.Cu at (104.5, 103.2)
- added kibuzzard-699C2DF3: G***, kibuzzard-699C2DF3, F.Cu at (79.2, 137.8)
- added kibuzzard-699C2E08: G***, kibuzzard-699C2E08, F.Cu at (93.9, 137.8)
- added kibuzzard-699C2E08: G***, kibuzzard-699C2E08, F.Cu at (108.5, 137.8)
- added kibuzzard-699C2E52: G***, kibuzzard-699C2E52, F.Cu at (64.5, 137.8)
- added kibuzzard-699C2E8F: G***, kibuzzard-699C2E8F, F.Cu at (35.4, 145.4)
- added kibuzzard-699C2EC2: G***, kibuzzard-699C2EC2, F.Cu at (50.0, 145.4)
- added kibuzzard-699C2EF8: G***, kibuzzard-699C2EF8, F.Cu at (46.0, 148.9)
- added kibuzzard-699C2F02: G***, kibuzzard-699C2F02, F.Cu at (46.0, 152.7)
- added kibuzzard-699C2F1B: G***, kibuzzard-699C2F1B, F.Cu at (75.3, 141.3)
- added kibuzzard-699C2F31: G***, kibuzzard-699C2F31, F.Cu at (75.3, 145.0)
- added kibuzzard-699C2F5C: G***, kibuzzard-699C2F5C, F.Cu at (89.9, 141.3)
- added kibuzzard-699C2F61: G***, kibuzzard-699C2F61, F.Cu at (89.9, 145.1)
- added kibuzzard-699C2F67: G***, kibuzzard-699C2F67, F.Cu at (104.5, 140.6)
- added kibuzzard-699C2F70: G***, kibuzzard-699C2F70, F.Cu at (104.5, 145.1)
- added kibuzzard-699C2F7D: G***, kibuzzard-699C2F7D, F.Cu at (75.2, 148.9)
- added kibuzzard-699C2F83: G***, kibuzzard-699C2F83, F.Cu at (75.2, 152.7)
- added kibuzzard-699C2F89: G***, kibuzzard-699C2F89, F.Cu at (89.7, 148.9)
- added kibuzzard-699C2F8F: G***, kibuzzard-699C2F8F, F.Cu at (89.8, 152.7)
- added kibuzzard-699C2F95: G***, kibuzzard-699C2F95, F.Cu at (104.4, 148.9)
- added kibuzzard-699C2F9C: G***, kibuzzard-699C2F9C, F.Cu at (104.4, 152.7)
- added kibuzzard-699C2FA4: G***, kibuzzard-699C2FA4, F.Cu at (104.4, 133.0)
- added kibuzzard-699C2FB0: G***, kibuzzard-699C2FB0, F.Cu at (104.4, 131.1)
- C2: footprint Capacitor_SMD:C_0805_2012Metric -> Capacitor_SMD:C_0603_1608Metric
- C8: value 68µF/16V -> 10µF/25V; footprint Capacitor_Tantalum_SMD:CP_EIA-7343-43_Kemet-X -> Capacitor_SMD:C_0603_1608Metric
- moved J3 65.9 mm to (112.1, 133.0)
- moved kibuzzard-6985F394 59.7 mm to (111.9, 125.8)
- moved R3 49.3 mm to (110.2, 98.1)
- moved kibuzzard-6985EF84 15.7 mm to (60.6, 143.1)
- moved kibuzzard-6985EF8A 14.7 mm to (60.6, 150.8)
- moved U4 8.26 mm to (129.9, 114.0), turned to 90 degrees
- moved D6 7.30 mm to (108.6, 141.9)
- moved D7 7.30 mm to (108.6, 144.5)
- moved C5 5.08 mm to (128.6, 99.4)
- moved JP1 5.08 mm to (124.8, 100.6)
- moved JP2 5.08 mm to (124.8, 98.1)
- moved JP5 5.08 mm to (124.8, 105.7)
- moved U1 5.08 mm to (124.8, 99.4)
- moved kibuzzard-6985F567 5.08 mm to (124.8, 95.9)
- moved kibuzzard-6985F5B0 5.08 mm to (124.8, 103.5)
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Connections:
- C8 pad 1: +5V -> GND
- C8 pad 2: GND -> +5V
- R4 pad 2: Net-(JP3-A) -> D1/SCL
- R5 pad 2: Net-(JP4-A) -> D2/SDA
Routing:
- net +3.3V: track 5.33 -> 154.5 mm, vias 8 -> 10
- net +9V: track 0.00 -> 75.4 mm, vias 11 -> 0
- net En Motor: track 63.6 -> 2.35 mm
- net NEUT: track 0.00 -> 55.9 mm
- net Net-(S1-+LED): track 15.5 -> 59.4 mm, vias 0 -> 1
- net Net-(BT1-+): track 0.00 -> 36.9 mm, vias 0 -> 2
- net Net-(PS1-LINE): track 0.00 -> 32.9 mm
- net RX: track 95.1 -> 76.0 mm, vias 0 -> 2
- net LINE: track 0.00 -> 18.4 mm
- net TX: track 82.3 -> 64.3 mm, vias 0 -> 2
- net +5V: track 19.6 -> 31.8 mm, vias 1 -> 0
- net D3/TX1: track 93.0 -> 82.7 mm
- net D2/SDA: track 85.4 -> 93.5 mm, vias 0 -> 1
- net 230V Motor: track 0.00 -> 6.35 mm
- net D1/SCL: track 84.9 -> 91.2 mm, vias 0 -> 1
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- added copper zone on F.Cu, net +3.3V
- added copper zone on In1.Cu, net GND
- added copper zone on In2.Cu, net GND
- removed copper zone on In2.Cu, net +3.3V
- removed copper zone on In1.Cu, net +5V
- removed copper zone on In1.Cu, net +9V
Other:
- outline, holes or cut-outs redrawn

Commit message: bxcbxc
Parts:
- removed BT1: Battery_Cell, Battery:BatteryHolder_Keystone_3034_1x20mm
- removed C1: 15µF/50V, Capacitor_Tantalum_SMD:CP_EIA-7343-43_Kemet-X
- removed C2: 10nF/50V, Capacitor_SMD:C_0603_1608Metric
- removed C3: 68µF/16V, Capacitor_Tantalum_SMD:CP_EIA-7343-43_Kemet-X
- removed C6: 100nF/50V, Capacitor_SMD:C_0603_1608Metric
- removed C7: 1µF/50V, Capacitor_SMD:C_0603_1608Metric
- removed C8, C9: 10µF/25V, Capacitor_SMD:C_0603_1608Metric
- removed D1: SS14, Diode_SMD:D_SMA
- removed D2, D3, D4, D5, D6, D7, D8, D9: LESD5D5.0CT1G, Diode_SMD:D_SOD-523
- removed DRA1, DRA2: DIN_Rail_Adapter, MountingEquipment:DINRailAdapter_3xM3_PhoenixContact_1201578
- removed J3: VDD, Connector_Phoenix_MC:PhoenixContact_MCV_1,5_2-G-3.81_1x02_P3.81mm_Vertical
- removed J4: D5 & D6, Connector_Phoenix_MC:PhoenixContact_MCV_1,5_4-G-3.81_1x04_P3.81mm_Vertical
- removed JP1, JP5: RX Select, Jumper:SolderJumper-3_P1.3mm_Open_Pad1.0x1.5mm
- removed JP2: TX Select, Jumper:SolderJumper-3_P1.3mm_Open_Pad1.0x1.5mm
- removed L1: 33µH, Inductor_SMD:L_Chilisin_BMRB00060650
- removed U5: DS3231MZ, Package_SO:SOIC-8_3.9x4.9mm_P1.27mm
- removed kibuzzard-6985EF84: G***, kibuzzard-6985EF84
- removed kibuzzard-6985EF8A: G***, kibuzzard-6985EF8A
- removed kibuzzard-6985F394: G***, kibuzzard-6985F394
- removed kibuzzard-6985F472: G***, kibuzzard-6985F472
- removed kibuzzard-6985F4E1: G***, kibuzzard-6985F4E1
- removed kibuzzard-6985F4F7: G***, kibuzzard-6985F4F7
- removed kibuzzard-6985F567: G***, kibuzzard-6985F567
- removed kibuzzard-6985F5B0: G***, kibuzzard-6985F5B0
- removed kibuzzard-6985F603: G***, kibuzzard-6985F603
- removed kibuzzard-6985F68A: G***, kibuzzard-6985F68A
- removed the kibuzzard-699C2E08 at (108.5, 137.8)
- removed kibuzzard-699C2E8F: G***, kibuzzard-699C2E8F
- removed kibuzzard-699C2EC2: G***, kibuzzard-699C2EC2
- removed kibuzzard-699C2F1B: G***, kibuzzard-699C2F1B
- removed kibuzzard-699C2F31: G***, kibuzzard-699C2F31
- removed kibuzzard-699C2F5C: G***, kibuzzard-699C2F5C
- removed kibuzzard-699C2F61: G***, kibuzzard-699C2F61
- removed kibuzzard-699C2F67: G***, kibuzzard-699C2F67
- removed kibuzzard-699C2F70: G***, kibuzzard-699C2F70
- removed kibuzzard-699C2F7D: G***, kibuzzard-699C2F7D
- removed kibuzzard-699C2F83: G***, kibuzzard-699C2F83
- removed kibuzzard-699C2F89: G***, kibuzzard-699C2F89
- removed kibuzzard-699C2F8F: G***, kibuzzard-699C2F8F
- removed kibuzzard-699C2F95: G***, kibuzzard-699C2F95
- removed kibuzzard-699C2F9C: G***, kibuzzard-699C2F9C
- removed kibuzzard-699C2FA4: G***, kibuzzard-699C2FA4
- removed kibuzzard-699C2FB0: G***, kibuzzard-699C2FB0
- added kibuzzard-69B3E2B0: G***, kibuzzard-69B3E2B0, F.Cu at (31.4, 152.1)
- added kibuzzard-69B3E2CA: G***, kibuzzard-69B3E2CA, F.Cu at (31.4, 141.9)
- added kibuzzard-69B3E350: G***, kibuzzard-69B3E350, F.Cu at (61.0, 146.0)
- added kibuzzard-69B3E357: G***, kibuzzard-69B3E357, F.Cu at (61.0, 153.7)
- added kibuzzard-69B3E35C: G***, kibuzzard-69B3E35C, F.Cu at (76.0, 144.1)
- added kibuzzard-69B3E365: G***, kibuzzard-69B3E365, F.Cu at (76.0, 147.9)
- added kibuzzard-69B3E36A: G***, kibuzzard-69B3E36A, F.Cu at (75.9, 151.8)
- added kibuzzard-69B3E36E: G***, kibuzzard-69B3E36E, F.Cu at (75.9, 155.5)
- added kibuzzard-69B3E379: G***, kibuzzard-69B3E379, F.Cu at (90.6, 144.1)
- added kibuzzard-69B3E37F: G***, kibuzzard-69B3E37F, F.Cu at (90.6, 147.9)
- added kibuzzard-69B3E384: G***, kibuzzard-69B3E384, F.Cu at (90.5, 151.8)
- added kibuzzard-69B3E389: G***, kibuzzard-69B3E389, F.Cu at (90.5, 155.6)
- C4, C5: value 100nF/50V -> 100nF/25V
- J1: footprint Connector_Phoenix_MC:PhoenixContact_MCV_1,5_2-G-3.81_1x02_P3.81mm_Vertical -> Connector_Phoenix_MSTB:PhoenixContact_MSTBVA_2,5_4-G-5,08_1x04_P5.08mm_Vertical
- J2: value Mains Motor -> Conn_02x04_Odd_Even; footprint Connector_Phoenix_MC:PhoenixContact_MCV_1,5_2-G-3.81_1x02_P3.81mm_Vertical -> Connector_PinSocket_2.54mm:PinSocket_2x04_P2.54mm_Horizontal
- R3: value 100R -> 330R
- U2: value LM2675M-3.3 -> TSR3-2433N; footprint Package_SO:SOIC-8_3.9x4.9mm_P1.27mm -> Converter_DCDC:Converter_DCDC_TRACO_TSR2-24xxN_TSR2-24xxxN_THT; moved to F.Cu
- U3: value WEMOS_D1_mini -> ESP32-S3-ZERO; footprint RF_Module:WEMOS_D1_mini_light -> lib:ESP32-S3-ZERO
- U4: value NCP1117-5.0_SOT223 -> TSR3-2450N; footprint Package_TO_SOT_SMD:SOT-223-3_TabPin2 -> Converter_DCDC:Converter_DCDC_TRACO_TSR2-24xxN_TSR2-24xxxN_THT; moved to F.Cu
- moved J2 69.9 mm to (117.2, 123.5), turned to 180 degrees
- moved U4 38.0 mm to (97.8, 134.3), turned to -90 degrees
- moved R4 26.3 mm to (107.6, 105.1)
- moved R5 25.5 mm to (107.6, 102.5)
- moved C5 17.7 mm to (114.6, 110.2), turned to 90 degrees
- moved kibuzzard-699C2EF8 15.7 mm to (31.4, 154.6)
- moved U2 15.3 mm to (82.2, 134.3), turned to -90 degrees
- moved kibuzzard-699C2F02 14.9 mm to (31.4, 149.5)
- moved kibuzzard-6985EF62 13.3 mm to (31.4, 139.4)
- moved F2 12.6 mm to (50.2, 154.6)
- moved U1 12.5 mm to (118.4, 110.2), turned to 0 degrees
- moved J8 12.4 mm to (111.4, 130.2)
- moved J9 12.4 mm to (121.6, 130.2)
- moved F1 11.3 mm to (50.2, 144.5)
- moved C4 10.9 mm to (122.2, 110.2), turned to 90 degrees
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Connections:
- J1 pad 1: NEUT -> 230V Motor
- J1 pad 2: LINE -> NEUT
- J10 pad 3: D2/SDA -> SDA
- J10 pad 4: D1/SCL -> SCL
- J11 pad 3: D4/RX1 -> GPIO1
- J11 pad 4: D3/TX1 -> GPIO2
- J2 pad 1: NEUT -> +9V
- J2 pad 2: 230V Motor -> +9V
- R4 pad 2: D1/SCL -> SCL
- R5 pad 2: D2/SDA -> SDA
- U1 pad 4: TX Selected -> TX_
- U1 pad 5: RX Selected -> RX_
- U1 pad 6: OE -> +3.3V
- U2 pad 1: /CB -> +9V
- U2 pad 2: unconnected-(U2-NC-Pad2) -> GND
- U2 pad 3: unconnected-(U2-NC-Pad3) -> +3.3V
- U3 pad 1: unconnected-(U3-~{RST}-Pad1) -> GPIO1
- U3 pad 10: GND -> unconnected-(U3-GP10-Pad10)
- U3 pad 11: D4/RX1 -> En Motor
- U3 pad 12: D3/TX1 -> SDA
- U3 pad 13: D2/SDA -> SCL
- U3 pad 2: unconnected-(U3-A0-Pad2) -> GPIO2
- U3 pad 3: En Motor -> unconnected-(U3-GP3-Pad3)
- U3 pad 4: D5 -> unconnected-(U3-GP4-Pad4)
- U3 pad 5: D6 -> unconnected-(U3-GP5-Pad5)
- U3 pad 6: Enable UART -> unconnected-(U3-GP6-Pad6)
- U3 pad 9: +5V -> unconnected-(U3-GP9-Pad9)
- U4 pad 1: GND -> +9V
- U4 pad 2: +5V -> GND
- U4 pad 3: +9V -> +5V
Routing:
- net +3.3V: track 154.5 -> 10.00 mm, vias 10 -> 2
- net SDA: track 0.00 -> 99.5 mm, vias 0 -> 1
- net D2/SDA: track 93.5 -> 0.00 mm, vias 1 -> 0
- net SCL: track 0.00 -> 92.7 mm, vias 0 -> 1
- net D1/SCL: track 91.2 -> 0.00 mm, vias 1 -> 0
- net D4/RX1: track 84.0 -> 0.00 mm
- net D3/TX1: track 82.7 -> 0.00 mm
- net GPIO1: track 0.00 -> 64.9 mm
- net GPIO2: track 0.00 -> 64.7 mm
- net D6: track 51.3 -> 0.00 mm
- net D5: track 48.4 -> 0.00 mm
- net Net-(BT1-+): track 36.9 -> 0.00 mm, vias 2 -> 0
- net +9V: track 75.4 -> 48.7 mm
- net +5V: track 31.8 -> 55.2 mm
- net RX: track 76.0 -> 55.4 mm, vias 2 -> 1
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- added copper zone on In1.Cu, net +3.3V
- added copper zone on In1.Cu, net +9V
- removed copper zone on B.Cu, net +3.3V
- removed copper zone on F.Cu, net +3.3V
- removed copper zone on B.Cu, net +9V
- removed copper zone on B.Cu, net /CB
- removed copper zone on B.Cu, net /VSW
- removed copper zone on In1.Cu, net GND
Other:
- board size 124.5 x 63.5 mm -> 100 x 72 mm
- board text removed: "espSFDmains"

Commit message: teruzrtu
Parts:
- added C1: 4.7µF 50V, Capacitor_SMD:C_0805_2012Metric, B.Cu at (82.2, 124.5)
- added C10: 10µF 25V, Capacitor_SMD:C_0805_2012Metric, B.Cu at (97.2, 132.7)
- added C2: 4.7µF 50V, Capacitor_SMD:C_0805_2012Metric, B.Cu at (77.8, 132.7)
- added C3: 10µF 25V, Capacitor_SMD:C_0805_2012Metric, B.Cu at (81.6, 132.7)
- added C8: 4.7µF 50V, Capacitor_SMD:C_0805_2012Metric, B.Cu at (96.5, 124.5)
- added C9: 4.7µF 50V, Capacitor_SMD:C_0805_2012Metric, B.Cu at (93.3, 132.7)
- added L1: 4,7µH 3A, Inductor_SMD:L_Sunlord_MWSA0402S, B.Cu at (78.4, 124.5)
- added L2: 4,7µH 3A, Inductor_SMD:L_Sunlord_MWSA0402S, B.Cu at (92.7, 124.5)
- J2: value Conn_02x04_Odd_Even -> Board Interconn; footprint Connector_PinSocket_2.54mm:PinSocket_2x04_P2.54mm_Horizontal -> Connector_PinSocket_1.27mm:PinSocket_2x09_P1.27mm_Horizontal
- moved U2 6.96 mm to (77.2, 129.5), turned to 90 degrees
- moved U4 6.96 mm to (92.7, 129.5), turned to 90 degrees
- moved J2 6.35 mm to (123.5, 123.5)
Connections:
- J2 pad 3: GND -> +9V
- J2 pad 4: GND -> +9V
- J2 pad 5: SCL -> GND
- J2 pad 7: SDA -> RX_
- U2 pad 1: +9V -> Net-(U2-Vin)
- U3 pad 3: unconnected-(U3-GP3-Pad3) -> GPIO3
- U3 pad 4: unconnected-(U3-GP4-Pad4) -> GPIO4
- U4 pad 1: +9V -> Net-(U4-Vin)
Routing:
- net GPIO4: track 0.00 -> 22.1 mm
- net RX_: track 10.8 -> 32.8 mm
- net GPIO3: track 0.00 -> 20.6 mm
- net +9V: track 48.7 -> 29.0 mm
- net En Motor: track 2.35 -> 21.5 mm
- net TX_: track 7.99 -> 23.5 mm
- net Net-(U2-Vin): track 0.00 -> 7.06 mm
- net Net-(U4-Vin): track 0.00 -> 6.54 mm
- net TX: track 53.5 -> 49.3 mm
- net Net-(S1-+LED): track 61.7 -> 58.8 mm
- net +3.3V: track 10.00 -> 12.7 mm
- net RX: track 55.4 -> 53.0 mm
- net GPIO2: track 64.7 -> 66.2 mm
- net +5V: track 55.2 -> 56.5 mm
- net SDA: track 99.5 -> 100.9 mm
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