File: hardware/pcb/espSFDmains/espSFDmains.kicad_sch (KiCad schematic)
At the start: 32 parts, among them J1 Mains, J10 D1 & D2, J11 D3 & D4, J2 Mains Motor, J3 VDD, J4 D5 & D6, J5 Motor, J8 SFD Bus, J9 SFD Bus, U1 TXS0102DCT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

Commit message: fhdgfh
Parts:
- added D2, D3, D4, D5, D6, D7, D8, D9: LESD5D5.0CT1G, Diode_SMD:D_SOD-523, symbol Device:D_TVS
- JP1: value SolderJumper_3_Open -> RX Select
- JP2: value SolderJumper_3_Open -> TX Select
Connections:
- net D1/SCL: now also D5.2 (A2)
- net D2/SDA: now also D2.2 (A2)
- net D3/TX1: now also D3.2 (A2)
- net D4/RX1: now also D4.2 (A2)
- net D5: now also D6.2 (A2)
- net D6: now also D7.2 (A2)
- net RX: now also D8.2 (A2)
- net TX: now also D9.2 (A2)
- net TX Selected: now reaches JP2.2 (C), U1.4 (A2)
- net VSW: now reaches C2.2, D1.1 (K), L1.1, U2.8 (VSW)
- net CB: now reaches C2.1, U2.1 (CB)
- net RX Selected: now reaches JP1.2 (C), U1.5 (A1)
- net VCC renamed +5V
- net VDD renamed +9V
- net VSS renamed GND
- net GND: now also D2.1 (A1), D3.1 (A1), D4.1 (A1), D5.1 (A1), D6.1 (A1), D7.1 (A1), D8.1 (A1), D9.1 (A1)
- no-connect marks 3 -> 4
Other:
- moved on the sheet: C2, C4, C5, D1, J10, J11, J4, JP1, JP2, U1, U3

Commit message: vncvn
Parts:
- added JP5: RX Select, Jumper:SolderJumper-3_P1.3mm_Open_Pad1.0x1.5mm, symbol Jumper:SolderJumper_3_Open
Connections:
- net +3.3V: now also JP5.1 (A)
- net D1/SCL: now also J10.4 (Pin_4); no longer J10.3 (Pin_3)
- net D2/SDA: now also J10.3 (Pin_3); no longer J10.4 (Pin_4)
- net D3/TX1: now also J11.4 (Pin_4); no longer J11.3 (Pin_3)
- net D4/RX1: now also J11.3 (Pin_3); no longer J11.4 (Pin_4)
- net D5: now also J4.4 (Pin_4); no longer J4.3 (Pin_3)
- net D6: now also J4.3 (Pin_3); no longer J4.4 (Pin_4)
- net Enable UART: now also JP5.3 (B); no longer U1.6 (OE)
- net Motor L: now also J5.1 (Pin_1), J5.2 (Pin_2); no longer J5.3 (Pin_3), J5.4 (Pin_4)
- net Motor N: now also J5.3 (Pin_3), J5.4 (Pin_4); no longer J5.1 (Pin_1), J5.2 (Pin_2)
- new net OE: JP5.2 (C), U1.6 (OE)
Changed lines of the file:
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@@
 	(global_label "D4/RX1"
 		(shape input)
-		(at 240.03 142.24 180)
+		(at 240.03 139.7 180)
 		(fields_autoplaced yes)
 		(effects
@@
 		)
 		(property "Intersheetrefs" "${INTERSHEET_REFS}"
-			(at 229.5458 142.24 0)
+			(at 229.5458 139.7 0)
 			(effects
 				(font
@@
 		)
 	)
+	(global_label "Enable UART"
+		(shape bidirectional)
+		(at 118.11 191.77 180)
+		(fields_autoplaced yes)
+		(effects
+			(font
+				(size 1.27 1.27)
+			)
+			(justify right)
+		)
+		(property "Intersheetrefs" "${INTERSHEET_REFS}"
+			(at 102.0394 191.77 0)
+			(effects
+				(font
+					(size 1.27 1.27)
+				)
+				(justify right)
+				(hide yes)
+			)
+		)
+	)
 	(global_label "D5"
 		(shape input)
-		(at 240.03 158.75 180)
+		(at 240.03 161.29 180)
 		(fields_autoplaced yes)
 		(effects
@@
 		)
 		(property "Intersheetrefs" "${INTERSHEET_REFS}"
-			(at 234.5653 158.75 0)
+			(at 234.5653 161.29 0)
 			(effects
 				(font
@@
 	(global_label "Motor N"
 		(shape output)
-		(at 72.39 30.48 270)
+		(at 78.74 30.48 270)
 		(fields_autoplaced yes)
 		(effects
@@
 		)
 		(property "Intersheetrefs" "${INTERSHEET_REFS}"
-			(at 72.39 41.0246 90)
+			(at 78.74 41.0246 90)
 			(effects
 				(font
@@
 	(global_label "D3/TX1"
 		(shape input)
-		(at 240.03 139.7 180)
+		(at 240.03 142.24 180)
 		(fields_autoplaced yes)
 		(effects
@@
 		)
 		(property "Intersheetrefs" "${INTERSHEET_REFS}"
-			(at 229.8482 139.7 0)
+			(at 229.8482 142.24 0)
 			(effects
 				(font
@@
 	(global_label "D2{slash}SDA"
 		(shape input)
-		(at 240.03 123.19 180)
+		(at 240.03 120.65 180)
 		(fields_autoplaced yes)
 		(effects
@@
 		)
 		(property "Intersheetrefs" "${INTERSHEET_REFS}"
-			(at 229.6667 123.19 0)
+			(at 229.6667 120.65 0)
 			(effects
 				(font
@@
 	(global_label "D1{slash}SCL"
 		(shape input)
-		(at 240.03 120.65 180)
+		(at 240.03 123.19 180)
 		(fields_autoplaced yes)
 		(effects
@@
 		)
 		(property "Intersheetrefs" "${INTERSHEET_REFS}"
-			(at 229.7272 120.65 0)
+			(at 229.7272 123.19 0)
 			(effects
 				(font
@@
 		)
 	)
+	(global_label "OE"
+		(shape input)
+		(at 123.19 195.58 0)
+		(fields_autoplaced yes)
+		(effects
+			(font
+				(size 1.27 1.27)
+			)
+			(justify left)
+		)
+		(property "Intersheetrefs" "${INTERSHEET_REFS}"
+			(at 128.6547 195.58 0)
+			(effects
+				(font
+					(size 1.27 1.27)
+				)
+				(justify left)
+				(hide yes)
+			)
+		)
+	)
 	(global_label "TX Selected"
 		(shape input)
@@
 	(global_label "D6"
 		(shape input)
-		(at 240.03 161.29 180)
+		(at 240.03 158.75 180)
 		(fields_autoplaced yes)
 		(effects
@@
 		)
 		(property "Intersheetrefs" "${INTERSHEET_REFS}"
-			(at 234.5653 161.29 0)
+			(at 234.5653 158.75 0)
 			(effects
 				(font
@@
 		)
 	)
-	(global_label "Enable UART"
+	(global_label "OE"
 		(shape input)
 		(at 170.18 140.97 0)
@@
 		)
 		(property "Intersheetrefs" "${INTERSHEET_REFS}"
-			(at 185.1393 140.97 0)
+			(at 175.6447 140.97 0)
 			(effects
 				(font
@@
 	(global_label "Motor L"
 		(shape output)
-		(at 77.47 30.48 270)
+		(at 73.66 30.48 270)
 		(fields_autoplaced yes)
 		(effects
@@
 		)
 		(property "Intersheetrefs" "${INTERSHEET_REFS}"
-			(at 77.47 40.7222 90)
+			(at 73.66 40.7222 90)
 			(effects
 				(font
@@
 	)
 	(symbol
+		(lib_id "Jumper:SolderJumper_3_Open")
+		(at 123.19 191.77 0)
+		(mirror y)
+		(unit 1)
+		(exclude_from_sim no)
+		(in_bom yes)
+		(on_board yes)
+		(dnp no)
+		(property "Reference" "JP5"
+			(at 123.19 185.42 0)
+			(effects
+				(font
+					(size 1.27 1.27)
+				)
+			)
+		)
+		(property "Value" "RX Select"
+			(at 123.19 187.96 0)
+			(effects
+				(font
+					(size 1.27 1.27)
+				)
+			)
+		)
+		(property "Footprint" "Jumper:SolderJumper-3_P1.3mm_Open_Pad1.0x1.5mm"
+			(at 123.19 191.77 0)
+			(effects
+				(font
+					(size 1.27 1.27)
+				)
+				(hide yes)
+			)
+		)
+		(property "Datasheet" "~"
+			(at 123.19 191.77 0)
+			(effects
+				(font
+					(size 1.27 1.27)
+				)
+				(hide yes)
+			)
+		)
+		(property "Description" ""
+			(at 123.19 191.77 0)
+			(effects
+				(font
+					(size 1.27 1.27)
+				)
+				(hide yes)
+			)
+		)
+		(pin "3"
+		)
+		(pin "2"
+		)
+		(pin "1"
+		)
+		(instances
+			(project "espSFDmains"
+				(path "/b4f72b7f-c57f-4eed-9610-6133338117bb"
+					(reference "JP5")
+					(unit 1)
+				)
+			)
+		)
+	)
+	(symbol
 		(lib_id "Device:D_TVS")
 		(at 267.97 130.81 0)
@@
 					(unit 1)
 				)
+			)
+		)
+	)
+	(symbol
+		(lib_id "power:+3.3V")
+		(at 128.27 191.77 270)
+		(mirror x)
+		(unit 1)
+		(exclude_from_sim no)
+		(in_bom yes)
+		(on_board yes)
+		(dnp no)
+		(fields_autoplaced yes)
+		(property "Reference" "#PWR041"
+			(at 124.46 191.77 0)
+			(effects
+				(font
+					(size 1.27 1.27)
+				)
+				(hide yes)
+			)
+		)
+		(property "Value" "+3.3V"
+			(at 132.08 191.7699 90)
+			(effects
+				(font
+					(size 1.27 1.27)
+				)
+				(justify left)
+			)
+		)
+		(property "Footprint" ""
+			(at 128.27 191.77 0)
+			(effects
+				(font
+					(size 1.27 1.27)
+				)
+				(hide yes)
+			)
+		)
+		(property "Datasheet" ""
+			(at 128.27 191.77 0)
+			(effects
+				(font
+					(size 1.27 1.27)
+				)
+				(hide yes)
+			)
+		)
+		(property "Description" "Power symbol creates a global label with name \"+3.3V\""
+			(at 128.27 191.77 0)
+			(effects
+				(font
+					(size 1.27 1.27)
+				)
+				(hide yes)
+			)
+		)
+		(pin "1"
+		)
+		(instances
+			(project "espSFDmains"
+				(path "/b4f72b7f-c57f-4eed-9610-6133338117bb"
+					(reference "#PWR041")
+					(unit 1)
+				)

Commit message: ffd hdf
Parts:
- added C6, C8: 68µF/16V, Capacitor_Tantalum_SMD:CP_EIA-7343-43_Kemet-X, symbol Device:C_Polarized
- added C7: 15µF/50V, Capacitor_Tantalum_SMD:CP_EIA-7343-43_Kemet-X, symbol Device:C_Polarized
- added U4: NCP1117-3.3_SOT223, Package_TO_SOT_SMD:SOT-223-3_TabPin2, symbol Regulator_Linear:NCP1117-3.3_SOT223
Connections:
- net +3.3V: now also J10.2 (Pin_2), J11.2 (Pin_2), J4.2 (Pin_2), C8.1, U4.2 (VO); no longer U3.8 (3V3)
- net +5V: now also C6.1, U4.3 (VI); no longer J10.2 (Pin_2), J11.2 (Pin_2), J4.2 (Pin_2)
- net +9V: now also C7.1
- net GND: now also C6.2, C7.2, C8.2, U4.1 (GND)
- no-connect marks 4 -> 5

Commit message: dgs
Parts:
- removed C6: 68µF/16V, Capacitor_Tantalum_SMD:CP_EIA-7343-43_Kemet-X, symbol Device:C_Polarized
- removed C7: 15µF/50V, Capacitor_Tantalum_SMD:CP_EIA-7343-43_Kemet-X, symbol Device:C_Polarized
- removed U2: LM2675N-5, Package_SO:SOIC-8_3.9x4.9mm_P1.27mm, symbol Regulator_Switching:LM2675N-5
- removed U4: NCP1117-3.3_SOT223, Package_TO_SOT_SMD:SOT-223-3_TabPin2, symbol Regulator_Linear:NCP1117-3.3_SOT223
- added U2: LM2675M-3.3, Package_SO:SOIC-8_3.9x4.9mm_P1.27mm, symbol Regulator_Switching:LM2675M-3.3
- added U4: NCP1117-5.0_SOT223, Package_TO_SOT_SMD:SOT-223-3_TabPin2, symbol Regulator_Linear:NCP1117-5.0_SOT223
Connections:
- net +3.3V: now also C3.1, L1.2, U2.4 (FB); no longer C8.1
- net +5V: now also C8.1, U4.2 (VO); no longer C3.1, L1.2
- net +9V: now also U2.7 (VIN), U4.3 (VI)
- net CB: now also U2.1 (CB)
- net GND: now also U2.6 (GND), U4.1 (GND)
- net VSW: now also U2.8 (VSW)

Commit message: fhgfds hds
Parts:
- removed PS2: HLK-30M09, Converter_ACDC:Converter_ACDC_Hi-Link_HLK-30Mxx, symbol Converter_ACDC:HLK-30M09
- added PS1: TPP_30-109-D, lib:TPP_30-109-D, symbol TPP_30-109-D:TPP_30-109-D
Connections:
- net +9V: now also PS1.3 (+VOUT)
- net GND: now also PS1.4 (-VOUT)
- net NEUT: now also PS1.1 (NEUTRAL)
- net at F1.2: now also PS1.2 (LINE)
Other:
- moved on the sheet: F1

Commit message: ffg dsfb
Parts:
- removed C8: 68µF/16V, Capacitor_Tantalum_SMD:CP_EIA-7343-43_Kemet-X, symbol Device:C_Polarized
- removed JP3, JP4: SolderJumper_2_Open, Jumper:SolderJumper-2_P1.3mm_Open_Pad1.0x1.5mm, symbol Jumper:SolderJumper_2_Open
- added BT1: Battery_Cell, Battery:BatteryHolder_Keystone_3034_1x20mm, symbol Device:Battery_Cell
- added C6: 100nF/50V, Capacitor_SMD:C_0603_1608Metric, symbol Device:C
- added C7: 1µF/50V, Capacitor_SMD:C_0603_1608Metric, symbol Device:C
- added C8, C9: 10µF/25V, Capacitor_SMD:C_0603_1608Metric, symbol Device:C
- added U5: DS3231MZ, Package_SO:SOIC-8_3.9x4.9mm_P1.27mm, symbol Timer_RTC:DS3231MZ
- C2: footprint Capacitor_SMD:C_0805_2012Metric -> Capacitor_SMD:C_0603_1608Metric
Connections:
- net +3.3V: now also C6.2, C7.2, U5.2 (VCC)
- net +5V: now also C8.2
- net +9V: now also C9.2
- net D1/SCL: now also R4.2, U5.8 (SCL)
- net D2/SDA: now also R5.2, U5.7 (SDA)
- net GND: now also BT1.2 (-), C6.1, C7.1, C8.1, C9.1, U5.5 (GND)
- new net: BT1.1 (+), U5.6 (VBAT)
- no-connect marks 5 -> 8
Other:
- moved on the sheet: C4, C5, JP1, JP2, JP5, U1, U3

Commit message: bxcbxc
Parts:
- removed C1: 15µF/50V, Capacitor_Tantalum_SMD:CP_EIA-7343-43_Kemet-X, symbol Device:C_Polarized
- removed C2: 10nF/50V, Capacitor_SMD:C_0603_1608Metric, symbol Device:C
- removed C3: 68µF/16V, Capacitor_Tantalum_SMD:CP_EIA-7343-43_Kemet-X, symbol Device:C_Polarized
- removed C8, C9: 10µF/25V, Capacitor_SMD:C_0603_1608Metric, symbol Device:C
- removed D1: SS14, Diode_SMD:D_SMA, symbol Diode:SS14
- removed D2, D3, D4, D5, D6, D7, D8, D9: LESD5D5.0CT1G, Diode_SMD:D_SOD-523, symbol Device:D_TVS
- removed DRA1, DRA2: DIN_Rail_Adapter, MountingEquipment:DINRailAdapter_3xM3_PhoenixContact_1201578, symbol Mechanical:DIN_Rail_Adapter
- removed J2: Mains Motor, Connector_Phoenix_MC:PhoenixContact_MCV_1,5_2-G-3.81_1x02_P3.81mm_Vertical, symbol Connector:Conn_01x02_Socket
- removed J3: VDD, Connector_Phoenix_MC:PhoenixContact_MCV_1,5_2-G-3.81_1x02_P3.81mm_Vertical, symbol Connector:Conn_01x02_Socket
- removed J4: D5 & D6, Connector_Phoenix_MC:PhoenixContact_MCV_1,5_4-G-3.81_1x04_P3.81mm_Vertical, symbol Connector:Conn_01x04_Socket
- removed JP1, JP5: RX Select, Jumper:SolderJumper-3_P1.3mm_Open_Pad1.0x1.5mm, symbol Jumper:SolderJumper_3_Open
- removed JP2: TX Select, Jumper:SolderJumper-3_P1.3mm_Open_Pad1.0x1.5mm, symbol Jumper:SolderJumper_3_Open
- removed L1: 33µH, Inductor_SMD:L_Chilisin_BMRB00060650, symbol Device:L
- removed U2: LM2675M-3.3, Package_SO:SOIC-8_3.9x4.9mm_P1.27mm, symbol Regulator_Switching:LM2675M-3.3
- removed U3: WEMOS_D1_mini, RF_Module:WEMOS_D1_mini_light, symbol RF_Module:WEMOS_D1_mini
- removed U4: NCP1117-5.0_SOT223, Package_TO_SOT_SMD:SOT-223-3_TabPin2, symbol Regulator_Linear:NCP1117-5.0_SOT223
- added J2: Conn_02x04_Odd_Even, Connector_PinSocket_2.54mm:PinSocket_2x04_P2.54mm_Horizontal, symbol Connector_Generic:Conn_02x04_Odd_Even
- added U2: TSR3-2433N, Converter_DCDC:Converter_DCDC_TRACO_TSR2-24xxN_TSR2-24xxxN_THT, symbol Converter_DCDC:TSR3-2433N
- added U3: ESP32-S3-ZERO, lib:ESP32-S3-ZERO, symbol ESP32-S3-ZERO:ESP32-S3-ZERO
- added U4: TSR3-2450N, Converter_DCDC:Converter_DCDC_TRACO_TSR2-24xxN_TSR2-24xxxN_THT, symbol Converter_DCDC:TSR3-2450N
- BT1: JLCPCB Part # (none) -> C5213768; now left out of the parts list
- C4, C5: value 100nF/50V -> 100nF/25V; JLCPCB Part # C326783 -> C14663
- C6: value 100nF/50V -> 100nF/25V; JLCPCB Part # C326783 -> C14663; now left out of the parts list
- C7: JLCPCB Part # C326783 -> C15849; now left out of the parts list
- J1: footprint Connector_Phoenix_MC:PhoenixContact_MCV_1,5_2-G-3.81_1x02_P3.81mm_Vertical -> Connector_Phoenix_MSTB:PhoenixContact_MSTBVA_2,5_4-G-5,08_1x04_P5.08mm_Vertical; symbol Connector:Conn_01x02_Socket -> Connector:Conn_01x04_Socket
- R3: value 100R -> 330R; JLCPCB Part # (none) -> C22775
- R4, R5: JLCPCB Part # (none) -> C23162
- U1: JLCPCB Part # (none) -> C324082
- U5: JLCPCB Part # (none) -> C107410; now left out of the parts list
Connections:
- net OE is gone; now on net +3.3V: U1.6 (OE)
- net +3.3V: now also U2.3 (Vout)
- net +5V: now also U3.5V, U4.3 (Vout)
- net +9V: now also J2.1 (Pin_1), J2.2 (Pin_2), U2.1 (Vin), U4.1 (Vin)
- net 230V Motor: now also J1.1 (Pin_1)
- net En Motor: now also U3.11 (GP11)
- net GND: now also J2.3 (Pin_3), J2.4 (Pin_4), J2.6 (Pin_6), J2.8 (Pin_8), U2.2 (GND), U3.GND, U4.2 (GND)
- net LINE: now also J1.3 (Pin_3); no longer J1.2 (Pin_2)
- net NEUT: now also J1.2 (Pin_2), J1.4 (Pin_4); no longer J1.1 (Pin_1)
- net D1/SCL renamed SCL
- net SCL: now also J2.5 (Pin_5), U3.13 (GP13)
- net D2/SDA renamed SDA
- net SDA: now also J2.7 (Pin_7), U3.12 (GP12)
- net D3/TX1 renamed GPIO2
- net GPIO2: now also U3.2 (GP2)
- net D4/RX1 renamed GPIO1
- net GPIO1: now also U3.1 (GP1)
- net RX Selected renamed RX_
- net RX_: now also U3.RX
- net TX Selected renamed TX_
- net TX_: now also U3.TX
- no-connect marks 8 -> 4
