File: hardware/pcb/espSFDmains/espSFDmains.kicad_sch (KiCad schematic)
At the start: 24 parts, among them J1 Mains, J10 D1 & D2, J11 D3 & D4, J2 Conn_02x04_Odd_Even, J5 Motor, J8 SFD Bus, J9 SFD Bus, U1 TXS0102DCT, U2 TSR3-2433N, U3 ESP32-S3-ZERO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

Commit message: teruzrtu
Parts:
- added C1, C2, C8, C9: 4.7µF 50V, Capacitor_SMD:C_0805_2012Metric, symbol Device:C_Small
- added C10, C3: 10µF 25V, Capacitor_SMD:C_0805_2012Metric, symbol Device:C_Small
- added L1, L2: 4,7µH 3A, Inductor_SMD:L_Sunlord_MWSA0402S, symbol Device:L_Small
- J2: value Conn_02x04_Odd_Even -> Board Interconn; footprint Connector_PinSocket_2.54mm:PinSocket_2x04_P2.54mm_Horizontal -> Connector_PinSocket_1.27mm:PinSocket_2x09_P1.27mm_Horizontal; symbol Connector_Generic:Conn_02x04_Odd_Even -> Connector_Generic:Conn_02x09_Odd_Even
Connections:
- net +3.3V: now also C3.2
- net +5V: now also C10.2
- net +9V: now also J2.3 (Pin_3), J2.4 (Pin_4), C1.2, C8.2, L1.1, L2.1; no longer U2.1 (Vin), U4.1 (Vin)
- net En Motor: now also J2.17 (Pin_17)
- net GND: now also J2.10 (Pin_10), J2.12 (Pin_12), J2.14 (Pin_14), J2.15 (Pin_15), J2.5 (Pin_5), C1.1, C10.1, C2.1, C3.1, C8.1, C9.1; no longer J2.3 (Pin_3), J2.4 (Pin_4)
- net RX_: now also J2.7 (Pin_7)
- net SCL: now also J2.11 (Pin_11); no longer J2.5 (Pin_5)
- net SDA: now also J2.13 (Pin_13); no longer J2.7 (Pin_7)
- net TX_: now also J2.9 (Pin_9)
- net GPIO3: now reaches U3.3 (GP3)
- net GPIO3: now also J2.16 (Pin_16)
- net GPIO4: now reaches U3.4 (GP4)
- net GPIO4: now also J2.18 (Pin_18)
- new net: C2.2, L1.2, U2.1 (Vin)
- new net: C9.2, L2.2, U4.1 (Vin)
Other:
- moved on the sheet: U2, U4
